Commit message: add wheel macro do common

File: urdf/quimera.urdf.xacro (robot description, xacro)
@@ -1,4 +1,11 @@
 <?xml version="1.0"?>
 <robot xmlns:xacro="http://www.ros.org/wiki/xacro" name="mobile_robot">
+  <xacro:include filename="$(find quimera_robot_description)/urdf/common_macro.xacro" />
+  <xacro:property name="yaml" value="$(find quimera_robot_description)/config/wheel.yaml" />
+  <xacro:property name="wheel_props" value="${load_yaml(yaml)}"/>
+  <xacro:property name="front_wheel_yaml" value="$(find quimera_robot_description)/config/front_wheel.yaml" />
+  <xacro:property name="front_wheel_props" value="${load_yaml(front_wheel_yaml)}"/>
+  <xacro:property name="base_yaml" value="$(find quimera_robot_description)/config/base.yaml" />
+  <xacro:property name="base_props" value="${load_yaml(base_yaml)}"/>
   <xacro:property name="PI" value="3.14"/>
   <xacro:property name="base_width" value="0.198"/>
@@ -30,42 +37,4 @@
   <xacro:property name="caster_pos_y_joint" value="${(base_width/2) - caster_y_offset - (caster_height/2)}"/>
   <xacro:property name="caster_pos_z_joint" value="${caster_z_offset}"/>
-  <!--Color Properties-->
-  <material name="blue">
-    <color rgba="0 0 0.8 1"/>
-  </material>
-  <material name="black">
-    <color rgba="0 0 0 1"/>
-  </material>
-  <material name="white">
-    <color rgba="1 1 1 1"/>
-  </material>
-  <material name="red">
-    <color rgba="0.8 0.0 0.0 1.0"/>
-  </material>
-  <!--Interial macros-->
-  <xacro:macro name="cylinder_inertia" params="m r h">
-    <inertial>
-      <mass value="${m}"/>
-      <inertia ixx="${m*(3*r*r+h*h)/12}" ixy = "0" ixz = "0" iyy="${m*(3*r*r+h*h)/12}" iyz = "0" izz="${m*r*r/2}"/>
-    </inertial>
-  </xacro:macro>
-  <xacro:macro name="box_inertia" params="m w h d">
-    <inertial>
-      <mass value="${m}"/>
-      <inertia ixx="${m / 12.0 * (d*d + h*h)}" ixy="0.0" ixz="0.0" iyy="${m / 12.0 * (w*w + h*h)}" iyz="0.0" izz="${m / 12.0 * (w*w + d*d)}"/>
-    </inertial>
-  </xacro:macro>
-  <xacro:macro name="sphere_inertia" params="m r">
-    <inertial>
-      <mass value="${m}"/>
-      <inertia ixx="${2.0*m*(r*r)/5.0}" ixy="0.0" ixz="0.0" iyy="${2.0*m*(r*r)/5.0}" iyz="0.0" izz="${2.0*m*(r*r)/5.0}"/>
-    </inertial>
-  </xacro:macro>
-  <xacro:macro name="default_inertial" params="mass">
-    <inertial>
-      <mass value="${mass}"/>
-      <inertia ixx="1.0" ixy="0.0" ixz="0.0" iyy="1.0" iyz="0.0" izz="1.0"/>
-    </inertial>
-  </xacro:macro>
   <!--Base link-->
   <link name="base_link">
@@ -84,59 +53,35 @@
     </collision>
   </link>
-  <!--Wheel link1 & joint macro-->
-  <xacro:macro name="wheel" params="prefix reflect pos_x_joint pos_y_joint pos_z_joint">
-    <link name="${prefix}_wheel">
-      <visual>
-        <origin xyz="0.0 0 0" rpy="${pi/2} 0 0"/>
-         <geometry>
-        <mesh filename="package://quimera_robot_description/meshes/wheel_2.dae" />
-      </geometry>
-        <material name="red"/>
-      </visual>
-      <collision>
-        <origin xyz="0 0 0" rpy="${pi/2} 0 0"/>
-        <geometry>
-          <cylinder radius="${main_wheel_radius}" length="0.005"/>
-        </geometry>
-      </collision>
-      <xacro:cylinder_inertia m="10" r="${main_wheel_radius}" h="0.005"/>
-    </link>
-    <joint name="${prefix}_wheel_joint" type="continuous">
-      <axis xyz="1 0 0" rpy="0 0 0" />
-      <parent link="base_link"/>
-      <child link="${prefix}_wheel"/>
-      <origin xyz="${pos_x_joint} ${reflect* pos_y_joint} ${pos_z_joint}" rpy="0 0 0"/>
-    </joint>
+<!--
+  <xacro:macro name="test" params="x">
+    <xacro:property name="posi_x" value="0.008 | ${x}"/>
   </xacro:macro>
-  <!--Wheel link1 & joint macro-->
-  <xacro:macro name="caster_wheel" params="prefix reflect pos_x_joint pos_y_joint pos_z_joint">
-    <link name="${prefix}_wheel">
-      <visual>
-        <origin xyz="0.0 0 0" rpy="${pi/2} 0 0"/>
-         <geometry>
-         <cylinder radius="${caster_radius}" length="0.005"/>
-        </geometry>
-        <material name="red"/>
-      </visual>
-      <collision>
-        <origin xyz="0 0 0" rpy="${pi/2} 0 0"/>
-        <geometry>
-          <cylinder radius="${caster_radius}" length="${caster_height}"/>
-        </geometry>
-      </collision>
-      <xacro:cylinder_inertia m="10" r="${caster_radius}" h="0.005"/>
-    </link>
-    <joint name="${prefix}_wheel_joint" type="continuous">
-      <axis xyz="1 0 0" rpy="0 0 0" />
-      <parent link="base_link"/>
-      <child link="${prefix}_wheel"/>
-      <origin xyz="${pos_x_joint} ${reflect* pos_y_joint} ${pos_z_joint}" rpy="0 0 0"/>
-    </joint>
-  </xacro:macro>
-  <!--Create Left & Right Wheel links/joints-->
-  <xacro:wheel prefix="left" reflect="1" pos_x_joint="${pos_x_joint}" pos_y_joint="${pos_y_joint}" pos_z_joint="${pos_z_joint}"/>
-  <xacro:wheel prefix="right" reflect="-1" pos_x_joint="${pos_x_joint}" pos_y_joint="${pos_y_joint}" pos_z_joint="${pos_z_joint}"/>
-  <xacro:caster_wheel prefix="caster_left" reflect="1" pos_x_joint="${caster_pos_x_joint}" pos_y_joint="${caster_pos_y_joint}" pos_z_joint="${caster_pos_z_joint}"/>
-  <xacro:caster_wheel prefix="caster_right" reflect="-1" pos_x_joint="${caster_pos_x_joint}" pos_y_joint="${caster_pos_y_joint}" pos_z_joint="${caster_pos_z_joint}"/>
+  <xacro:test x="2"/> -->
+  <xacro:wheel prefix="right" reflect="-1"
+                      wheel_prop="${wheel_props}"
+                      pos_x_joint="${pos_x_joint}"
+                      pos_y_joint="${pos_y_joint}"
+                      pos_z_joint="${pos_z_joint}"
+                      mesh="${wheel_props['wheel']['mesh']}">
+  </xacro:wheel>
+  <xacro:wheel prefix="left" reflect="1"
+                      wheel_prop="${wheel_props}"
+                      pos_x_joint="${pos_x_joint}"
+                      pos_y_joint="${pos_y_joint}"
+                      pos_z_joint="${pos_z_joint}"
+                      mesh="${wheel_props['wheel']['mesh']}">
+  </xacro:wheel>
+  <xacro:wheel prefix="caster_right" reflect="-1"
+                      wheel_prop="${front_wheel_props}"
+                      pos_x_joint="${caster_pos_x_joint}"
+                      pos_y_joint="${caster_pos_y_joint}"
+                      pos_z_joint="${caster_pos_z_joint}">
+  </xacro:wheel>
+  <xacro:wheel prefix="caster_left" reflect="1"
+                      wheel_prop="${front_wheel_props}"
+                      pos_x_joint="${caster_pos_x_joint}"
+                      pos_y_joint="${caster_pos_y_joint}"
+                      pos_z_joint="${caster_pos_z_joint}">
+  </xacro:wheel>
   <!-- <xacro:include filename="$(find mobile_description)/urdf/mobile_robot_gazebo_plugins.xacro"/>  -->
 </robot>

Commit message: Remove unecessary lines and add comments.

File: urdf/quimera.urdf.xacro (robot description, xacro)
@@ -9,7 +9,5 @@
   <xacro:property name="base_props" value="${load_yaml(base_yaml)}"/>
   <xacro:property name="PI" value="3.14"/>
-  <xacro:property name="main_wheel_radius" value="0.053"/>
-  <xacro:property name="main_wheel_height" value="0.033"/>
-  <xacro:property name="main_wheel_mass" value="0.27"/>
+  <!-- ####### Main Wheel Parameters ########## -->
   <!-- Offset distance from the outter border to the center of the wheel-->
   <xacro:property name="main_wheel_x_offset" value="0.128"/>
@@ -18,12 +16,12 @@
   <!-- Offset distance from the bottom border to the center of the wheel -->
   <xacro:property name="main_wheel_z_offset" value="0.05"/>
+  <!-- Main Wheel joint position -->
   <xacro:property name="pos_x_joint"
      value="${(base_props['base']['length']/2) - main_wheel_x_offset}"/>
   <xacro:property name="pos_y_joint"
-    value="${(base_props['base']['width']/2) - main_wheel_y_offset - (main_wheel_height/2)}"/>
+    value="${(base_props['base']['width']/2) - main_wheel_y_offset - (base_props['base']['height']/2)}"/>
   <xacro:property name="pos_z_joint" value="${main_wheel_z_offset}"/>
-  <xacro:property name="caster_radius" value="0.011"/>
-  <xacro:property name="caster_height" value="0.006"/>
-  <xacro:property name="caster_mass" value="0.01"/>
+  <!-- ######################################## -->
+  <!-- ####### Auxiliar Wheel Parameters ########## -->
   <!-- Offset distance from the outter border to the center of the wheel-->
   <xacro:property name="caster_x_offset" value="0.035"/>
@@ -32,8 +30,10 @@
   <!-- Offset distance from the bottom border to the center of the wheel -->
   <xacro:property name="caster_z_offset" value="0.008"/>
+  <!-- Main Wheel joint position -->
   <xacro:property name="caster_pos_x_joint" value="${(base_props['base']['length']/2) - caster_x_offset}"/>
   <xacro:property name="caster_pos_y_joint"
     value="${(base_props['base']['width']/2) - caster_y_offset - (base_props['base']['height']/2)}"/>
   <xacro:property name="caster_pos_z_joint" value="${caster_z_offset}"/>
+  <!-- ######################################## -->
   <!-- Base link -->
   <xacro:base base_prop="${base_props}" mesh="${base_props['base']['mesh']}" >
@@ -45,4 +45,5 @@
   </xacro:macro>
   <xacro:test x="2"/> -->
+  <!-- Main Wheel -->
   <xacro:wheel prefix="right" reflect="-1"
                       wheel_prop="${wheel_props}"
@@ -59,4 +60,5 @@
                       mesh="${wheel_props['wheel']['mesh']}">
   </xacro:wheel>
+  <!-- Auxiliar Wheel -->
   <xacro:wheel prefix="caster_right" reflect="-1"
                       wheel_prop="${front_wheel_props}"

Commit message: Correct joint positions and update yaml files.

File: urdf/quimera.urdf.xacro (robot description, xacro)
@@ -2,5 +2,5 @@
 <robot xmlns:xacro="http://www.ros.org/wiki/xacro" name="mobile_robot">
   <xacro:include filename="$(find quimera_robot_description)/urdf/common_macro.xacro" />
-  <xacro:property name="yaml" value="$(find quimera_robot_description)/config/wheel.yaml" />
+  <xacro:property name="yaml" value="$(find quimera_robot_description)/config/back_wheel.yaml" />
   <xacro:property name="wheel_props" value="${load_yaml(yaml)}"/>
   <xacro:property name="front_wheel_yaml" value="$(find quimera_robot_description)/config/front_wheel.yaml" />
@@ -20,5 +20,5 @@
      value="${(base_props['base']['length']/2) - main_wheel_x_offset}"/>
   <xacro:property name="pos_y_joint"
-    value="${(base_props['base']['width']/2) - main_wheel_y_offset - (base_props['base']['height']/2)}"/>
+    value="${(base_props['base']['width']/2) - main_wheel_y_offset - (wheel_props['wheel']['length']/2)}"/>
   <xacro:property name="pos_z_joint" value="${main_wheel_z_offset}"/>
   <!-- ######################################## -->
@@ -33,5 +33,5 @@
   <xacro:property name="caster_pos_x_joint" value="${(base_props['base']['length']/2) - caster_x_offset}"/>
   <xacro:property name="caster_pos_y_joint"
-    value="${(base_props['base']['width']/2) - caster_y_offset - (base_props['base']['height']/2)}"/>
+    value="${(base_props['base']['width']/2) - caster_y_offset - (front_wheel_props['wheel']['length']/2)}"/>
   <xacro:property name="caster_pos_z_joint" value="${caster_z_offset}"/>
   <!-- ######################################## -->

Commit message: Change wheel name reference for back and front.

File: urdf/quimera.urdf.xacro (robot description, xacro)
@@ -2,6 +2,6 @@
 <robot xmlns:xacro="http://www.ros.org/wiki/xacro" name="mobile_robot">
   <xacro:include filename="$(find quimera_robot_description)/urdf/common_macro.xacro" />
-  <xacro:property name="yaml" value="$(find quimera_robot_description)/config/back_wheel.yaml" />
-  <xacro:property name="wheel_props" value="${load_yaml(yaml)}"/>
+  <xacro:property name="back_wheel_yaml" value="$(find quimera_robot_description)/config/back_wheel.yaml" />
+  <xacro:property name="wheel_props" value="${load_yaml(back_wheel_yaml)}"/>
   <xacro:property name="front_wheel_yaml" value="$(find quimera_robot_description)/config/front_wheel.yaml" />
   <xacro:property name="front_wheel_props" value="${load_yaml(front_wheel_yaml)}"/>
@@ -9,30 +9,30 @@
   <xacro:property name="base_props" value="${load_yaml(base_yaml)}"/>
   <xacro:property name="PI" value="3.14"/>
-  <!-- ####### Main Wheel Parameters ########## -->
+  <!-- ####### Back Wheel Parameters ########## -->
   <!-- Offset distance from the outter border to the center of the wheel-->
-  <xacro:property name="main_wheel_x_offset" value="0.128"/>
+  <xacro:property name="b_wheel_x_offset" value="0.128"/>
   <!-- Offset distance from the outter border to the face of the wheel -->
-  <xacro:property name="main_wheel_y_offset" value="0.02"/>
+  <xacro:property name="b_wheel_y_offset" value="0.02"/>
   <!-- Offset distance from the bottom border to the center of the wheel -->
-  <xacro:property name="main_wheel_z_offset" value="0.05"/>
-  <!-- Main Wheel joint position -->
-  <xacro:property name="pos_x_joint"
-     value="${(base_props['base']['length']/2) - main_wheel_x_offset}"/>
-  <xacro:property name="pos_y_joint"
-    value="${(base_props['base']['width']/2) - main_wheel_y_offset - (wheel_props['wheel']['length']/2)}"/>
-  <xacro:property name="pos_z_joint" value="${main_wheel_z_offset}"/>
+  <xacro:property name="b_wheel_z_offset" value="0.05"/>
+  <!-- Back Wheel joint position -->
+  <xacro:property name="b_wheel_pos_x_joint"
+     value="${(base_props['base']['length']/2) - b_wheel_x_offset}"/>
+  <xacro:property name="b_wheel_pos_y_joint"
+    value="${(base_props['base']['width']/2) - b_wheel_y_offset - (wheel_props['wheel']['length']/2)}"/>
+  <xacro:property name="b_wheel_pos_z_joint" value="${b_wheel_z_offset}"/>
   <!-- ######################################## -->
-  <!-- ####### Auxiliar Wheel Parameters ########## -->
+  <!-- ####### Front Wheel Parameters ########## -->
   <!-- Offset distance from the outter border to the center of the wheel-->
-  <xacro:property name="caster_x_offset" value="0.035"/>
+  <xacro:property name="f_wheel_x_offset" value="0.035"/>
   <!-- Offset distance from the outter border to the face of the wheel -->
-  <xacro:property name="caster_y_offset" value="0.050"/>
+  <xacro:property name="f_wheel_y_offset" value="0.050"/>
   <!-- Offset distance from the bottom border to the center of the wheel -->
-  <xacro:property name="caster_z_offset" value="0.008"/>
-  <!-- Main Wheel joint position -->
-  <xacro:property name="caster_pos_x_joint" value="${(base_props['base']['length']/2) - caster_x_offset}"/>
-  <xacro:property name="caster_pos_y_joint"
-    value="${(base_props['base']['width']/2) - caster_y_offset - (front_wheel_props['wheel']['length']/2)}"/>
-  <xacro:property name="caster_pos_z_joint" value="${caster_z_offset}"/>
+  <xacro:property name="f_wheel_z_offset" value="0.008"/>
+  <!-- Front Wheel joint position -->
+  <xacro:property name="f_wheel_pos_x_joint" value="${(base_props['base']['length']/2) - f_wheel_x_offset}"/>
+  <xacro:property name="f_wheel_pos_y_joint"
+    value="${(base_props['base']['width']/2) - f_wheel_y_offset - (front_wheel_props['wheel']['length']/2)}"/>
+  <xacro:property name="f_wheel_pos_z_joint" value="${f_wheel_z_offset}"/>
   <!-- ######################################## -->
   <!-- Base link -->
@@ -45,31 +45,31 @@
   </xacro:macro>
   <xacro:test x="2"/> -->
-  <!-- Main Wheel -->
-  <xacro:wheel prefix="right" reflect="-1"
+  <!-- Back Wheel -->
+  <xacro:wheel prefix="back_right" reflect="-1"
                       wheel_prop="${wheel_props}"
-                      pos_x_joint="${pos_x_joint}"
-                      pos_y_joint="${pos_y_joint}"
-                      pos_z_joint="${pos_z_joint}"
+                      pos_x_joint="${b_wheel_pos_x_joint}"
+                      pos_y_joint="${b_wheel_pos_y_joint}"
+                      pos_z_joint="${b_wheel_pos_z_joint}"
                       mesh="${wheel_props['wheel']['mesh']}">
   </xacro:wheel>
-  <xacro:wheel prefix="left" reflect="1"
+  <xacro:wheel prefix="back_left" reflect="1"
                       wheel_prop="${wheel_props}"
-                      pos_x_joint="${pos_x_joint}"
-                      pos_y_joint="${pos_y_joint}"
-                      pos_z_joint="${pos_z_joint}"
+                      pos_x_joint="${b_wheel_pos_x_joint}"
+                      pos_y_joint="${b_wheel_pos_y_joint}"
+                      pos_z_joint="${b_wheel_pos_z_joint}"
                       mesh="${wheel_props['wheel']['mesh']}">
   </xacro:wheel>
-  <!-- Auxiliar Wheel -->
-  <xacro:wheel prefix="caster_right" reflect="-1"
+  <!-- Front Wheel -->
+  <xacro:wheel prefix="front_right" reflect="-1"
                       wheel_prop="${front_wheel_props}"
-                      pos_x_joint="${caster_pos_x_joint}"
-                      pos_y_joint="${caster_pos_y_joint}"
-                      pos_z_joint="${caster_pos_z_joint}">
+                      pos_x_joint="${f_wheel_pos_x_joint}"
+                      pos_y_joint="${f_wheel_pos_y_joint}"
+                      pos_z_joint="${f_wheel_pos_z_joint}">
   </xacro:wheel>
-  <xacro:wheel prefix="caster_left" reflect="1"
+  <xacro:wheel prefix="front_left" reflect="1"
                       wheel_prop="${front_wheel_props}"
-                      pos_x_joint="${caster_pos_x_joint}"
-                      pos_y_joint="${caster_pos_y_joint}"
-                      pos_z_joint="${caster_pos_z_joint}">
+                      pos_x_joint="${f_wheel_pos_x_joint}"
+                      pos_y_joint="${f_wheel_pos_y_joint}"
+                      pos_z_joint="${f_wheel_pos_z_joint}">
   </xacro:wheel>
   <!-- <xacro:include filename="$(find mobile_description)/urdf/mobile_robot_gazebo_plugins.xacro"/>  -->

Commit message: Change y joint position calculation and definition.

File: urdf/quimera.urdf.xacro (robot description, xacro)
@@ -12,6 +12,8 @@
   <!-- Offset distance from the outter border to the center of the wheel-->
   <xacro:property name="b_wheel_x_offset" value="0.128"/>
-  <!-- Offset distance from the outter border to the face of the wheel -->
-  <xacro:property name="b_wheel_y_offset" value="0.02"/>
+  <!-- Offset distance from the outer face of the base to the inner face of the wheel.
+   The outer face of the base is the reference so, if the wheels are inside the base the value must be
+   negative. If the wheels are outside, must be positive -->
+  <xacro:property name="b_wheel_y_offset" value="-0.052"/>
   <!-- Offset distance from the bottom border to the center of the wheel -->
   <xacro:property name="b_wheel_z_offset" value="0.05"/>
@@ -20,5 +22,5 @@
      value="${(base_props['base']['x_size']/2) - b_wheel_x_offset}"/>
   <xacro:property name="b_wheel_pos_y_joint"
-    value="${(base_props['base']['y_size']/2) - b_wheel_y_offset - (wheel_props['wheel']['length']/2)}"/>
+    value="${(base_props['base']['y_size']/2) + b_wheel_y_offset + (wheel_props['wheel']['length']/2)}"/>
   <xacro:property name="b_wheel_pos_z_joint" value="${b_wheel_z_offset}"/>
   <!-- ######################################## -->
@@ -26,6 +28,6 @@
   <!-- Offset distance from the outter border to the center of the wheel-->
   <xacro:property name="f_wheel_x_offset" value="0.035"/>
-  <!-- Offset distance from the outter border to the face of the wheel -->
-  <xacro:property name="f_wheel_y_offset" value="0.050"/>
+  <!-- Offset distance from the outter border of the base to the inner face of the wheel -->
+  <xacro:property name="f_wheel_y_offset" value="-0.056"/>
   <!-- Offset distance from the bottom border to the center of the wheel -->
   <xacro:property name="f_wheel_z_offset" value="0.008"/>
@@ -33,5 +35,5 @@
   <xacro:property name="f_wheel_pos_x_joint" value="${(base_props['base']['x_size']/2) - f_wheel_x_offset}"/>
   <xacro:property name="f_wheel_pos_y_joint"
-    value="${(base_props['base']['y_size']/2) - f_wheel_y_offset - (front_wheel_props['wheel']['length']/2)}"/>
+    value="${(base_props['base']['y_size']/2) + f_wheel_y_offset + (front_wheel_props['wheel']['length']/2)}"/>
   <xacro:property name="f_wheel_pos_z_joint" value="${f_wheel_z_offset}"/>
   <!-- ######################################## -->

Commit message: Change offset values as parameters at yaml file.

File: urdf/quimera.urdf.xacro (robot description, xacro)
@@ -9,32 +9,17 @@
   <xacro:property name="base_props" value="${load_yaml(base_yaml)}"/>
   <xacro:property name="PI" value="3.14"/>
-  <!-- ####### Back Wheel Parameters ########## -->
-  <!-- Offset distance from the outter border to the center of the wheel-->
-  <xacro:property name="b_wheel_x_offset" value="0.128"/>
-  <!-- Offset distance from the outer face of the base to the inner face of the wheel.
-   The outer face of the base is the reference so, if the wheels are inside the base the value must be
-   negative. If the wheels are outside, must be positive -->
-  <xacro:property name="b_wheel_y_offset" value="-0.052"/>
-  <!-- Offset distance from the bottom border to the center of the wheel -->
-  <xacro:property name="b_wheel_z_offset" value="0.05"/>
   <!-- Back Wheel joint position -->
   <xacro:property name="b_wheel_pos_x_joint"
-     value="${(base_props['base']['x_size']/2) - b_wheel_x_offset}"/>
+     value="${(base_props['base']['x_size']/2) - wheel_props['wheel']['x_offset']}"/>
   <xacro:property name="b_wheel_pos_y_joint"
-    value="${(base_props['base']['y_size']/2) + b_wheel_y_offset + (wheel_props['wheel']['length']/2)}"/>
-  <xacro:property name="b_wheel_pos_z_joint" value="${b_wheel_z_offset}"/>
+    value="${(base_props['base']['y_size']/2) + wheel_props['wheel']['y_offset'] + (wheel_props['wheel']['length']/2)}"/>
+  <xacro:property name="b_wheel_pos_z_joint" value="${wheel_props['wheel']['z_offset']}"/>
   <!-- ######################################## -->
-  <!-- ####### Front Wheel Parameters ########## -->
-  <!-- Offset distance from the outter border to the center of the wheel-->
-  <xacro:property name="f_wheel_x_offset" value="0.035"/>
-  <!-- Offset distance from the outter border of the base to the inner face of the wheel -->
-  <xacro:property name="f_wheel_y_offset" value="-0.056"/>
-  <!-- Offset distance from the bottom border to the center of the wheel -->
-  <xacro:property name="f_wheel_z_offset" value="0.008"/>
   <!-- Front Wheel joint position -->
-  <xacro:property name="f_wheel_pos_x_joint" value="${(base_props['base']['x_size']/2) - f_wheel_x_offset}"/>
+  <xacro:property name="f_wheel_pos_x_joint"
+    value="${(base_props['base']['x_size']/2) - front_wheel_props['wheel']['x_offset']}"/>
   <xacro:property name="f_wheel_pos_y_joint"
-    value="${(base_props['base']['y_size']/2) + f_wheel_y_offset + (front_wheel_props['wheel']['length']/2)}"/>
-  <xacro:property name="f_wheel_pos_z_joint" value="${f_wheel_z_offset}"/>
+    value="${(base_props['base']['y_size']/2) + front_wheel_props['wheel']['y_offset'] + (front_wheel_props['wheel']['length']/2)}"/>
+  <xacro:property name="f_wheel_pos_z_joint" value="${front_wheel_props['wheel']['z_offset']}"/>
   <!-- ######################################## -->
   <!-- <xacro:macro name="get_parameters" params="yaml_name prefix">
