Commit message: clean up the code

File: urdf/quimera.urdf.xacro (robot description, xacro)
@@ -29,11 +29,9 @@
   <!-- <xacro:get_parameters yaml_name="back_wheel" prefix="front"/> -->
   <!-- <xacro:property name="test_props" value="${props}"/> -->
-  <!-- <xacro:get_parameters yaml_name="front_wheel"/>
-  <xacro:property name="front_props" value="${props}"/> -->
   <!-- Base link -->
   <xacro:base base_prop="${base_props}" mesh="${base_props['base']['mesh']}" >
     <origin xyz="0 0 0" rpy="${PI/2} 0 -${PI/2}" />
   </xacro:base>
-  <!-- Back Wheel -->
+  <!-- Back Wheels -->
   <xacro:wheel prefix="back_right" reflect="-1"
                       wheel_prop="${wheel_props}"
@@ -50,5 +48,5 @@
                       mesh="${wheel_props['wheel']['mesh']}">
   </xacro:wheel>
-  <!-- Front Wheel -->
+  <!-- Front Wheels -->
   <xacro:wheel prefix="front_right" reflect="-1"
                       wheel_prop="${front_wheel_props}"
