Commit message: update inertia macros

File: urdf/common_macro.xacro (robot description, xacro)
@@ -32,5 +32,5 @@
       <xacro:cylinder_inertia m="${wheel_prop['wheel']['mass']}"
                               r="${wheel_prop['wheel']['radius']}"
-                              h="${wheel_prop['wheel']['length']}">
+                              l="${wheel_prop['wheel']['length']}">
       </xacro:cylinder_inertia>
     </link>
@@ -43,14 +43,17 @@
   </xacro:macro>
 <!--Intertial macros-->
-  <xacro:macro name="cylinder_inertia" params="m r h">
+  <xacro:macro name="cylinder_inertia" params="m r l">
     <inertial>
       <mass value="${m}"/>
-      <inertia ixx="${m*(3*r*r+h*h)/12}" ixy = "0" ixz = "0" iyy="${m*(3*r*r+h*h)/12}" iyz = "0" izz="${m*r*r/2}"/>
+      <inertia ixx="${m*(3*r*r+l*l)/12}" ixy = "0" ixz = "0"
+               iyy="${m*(3*r*r+l*l)/12}" iyz = "0" izz="${m*r*r/2}"/>
     </inertial>
   </xacro:macro>
-  <xacro:macro name="box_inertia" params="m w h d">
+ <xacro:macro name="box_inertia" params="m x y z">
     <inertial>
       <mass value="${m}"/>
-      <inertia ixx="${m / 12.0 * (d*d + h*h)}" ixy="0.0" ixz="0.0" iyy="${m / 12.0 * (w*w + h*h)}" iyz="0.0" izz="${m / 12.0 * (w*w + d*d)}"/>
+      <inertia ixx="${m / 12.0 * (y*y + z*z)}" ixy="0.0" ixz="0.0"
+               iyy="${m / 12.0 * (x*x + z*z)}" iyz="0.0"
+               izz="${m / 12.0 * (x*x + y*y)}"/>
     </inertial>
   </xacro:macro>

File: urdf/quimera.urdf.xacro (robot description, xacro)
@@ -39,5 +39,5 @@
   <!--Base link-->
   <link name="base_link">
-    <xacro:box_inertia m="10" w="${base_len}" h="${base_width}" d="0.01"/>
+    <xacro:box_inertia m="10" x="${base_len}" y="0.01" z="${base_width}" />
     <visual>
       <origin xyz="0 0 0" rpy="${PI/2} 0 -${PI/2}" />

Commit message: Add base macro

File: urdf/common_macro.xacro (robot description, xacro)
@@ -42,4 +42,38 @@
     </joint>
   </xacro:macro>
+<!--Base macro-->
+  <xacro:macro name="base"
+               params="base_prop mesh:='' *origin">
+    <link name="base_link">
+    <xacro:box_inertia m="${base_prop['base']['mass']}"
+                       x="${base_prop['base']['length']}"
+                       y="${base_prop['base']['width']}"
+                       z="${base_prop['base']['height']}">
+    </xacro:box_inertia>
+    <xacro:if value="${mesh != '' }" >
+      <visual>
+        <xacro:insert_block name="origin" />
+        <geometry>
+          <mesh filename="package://quimera_robot_description/meshes/${mesh}.dae" />
+        </geometry>
+        <material name="white" />
+      </visual>
+    </xacro:if>
+    <xacro:if value="${mesh == '' }" >
+      <visual>
+        <xacro:insert_block name="origin" />
+        <geometry>
+          <box size="${base_prop['base']['length']} ${base_prop['base']['width']} ${base_prop['base']['height']}"/>
+        </geometry>
+        <material name="white" />
+      </visual>
+    </xacro:if>
+    <collision>
+      <geometry>
+        <box size="${base_len} ${base_width} 0.01"/>
+      </geometry>
+    </collision>
+    </link>
+  </xacro:macro>
 <!--Intertial macros-->
   <xacro:macro name="cylinder_inertia" params="m r l">

File: urdf/quimera.urdf.xacro (robot description, xacro)
@@ -38,5 +38,5 @@
   <xacro:property name="caster_pos_z_joint" value="${caster_z_offset}"/>
   <!--Base link-->
-  <link name="base_link">
+  <!-- <link name="base_link">
     <xacro:box_inertia m="10" x="${base_len}" y="0.01" z="${base_width}" />
     <visual>
@@ -52,5 +52,8 @@
       </geometry>
     </collision>
-  </link>
+  </link> -->
+  <xacro:base base_prop="${base_props}" mesh="${base_props['base']['mesh']}" >
+    <origin xyz="0 0 0" rpy="${PI/2} 0 -${PI/2}" />
+  </xacro:base>
 <!--
   <xacro:macro name="test" params="x">

Commit message: Get base parameters from yaml file

File: urdf/common_macro.xacro (robot description, xacro)
@@ -71,5 +71,5 @@
     <collision>
       <geometry>
-        <box size="${base_len} ${base_width} 0.01"/>
+        <box size="${base_prop['base']['length']} ${base_prop['base']['width']} ${base_prop['base']['height']}"/>
       </geometry>
     </collision>

File: urdf/quimera.urdf.xacro (robot description, xacro)
@@ -9,8 +9,4 @@
   <xacro:property name="base_props" value="${load_yaml(base_yaml)}"/>
   <xacro:property name="PI" value="3.14"/>
-  <xacro:property name="base_width" value="0.198"/>
-  <xacro:property name="base_len" value="0.195"/>
-  <xacro:property name="base_height" value="0.182"/>
-  <xacro:property name="base_mass" value="2.5"/>
   <xacro:property name="main_wheel_radius" value="0.053"/>
   <xacro:property name="main_wheel_height" value="0.033"/>
@@ -22,6 +18,8 @@
   <!-- Offset distance from the bottom border to the center of the wheel -->
   <xacro:property name="main_wheel_z_offset" value="0.05"/>
-  <xacro:property name="pos_x_joint" value="${(base_len/2) - main_wheel_x_offset}"/>
-  <xacro:property name="pos_y_joint" value="${(base_width/2) - main_wheel_y_offset - (main_wheel_height/2)}"/>
+  <xacro:property name="pos_x_joint"
+     value="${(base_props['base']['length']/2) - main_wheel_x_offset}"/>
+  <xacro:property name="pos_y_joint"
+    value="${(base_props['base']['width']/2) - main_wheel_y_offset - (main_wheel_height/2)}"/>
   <xacro:property name="pos_z_joint" value="${main_wheel_z_offset}"/>
   <xacro:property name="caster_radius" value="0.011"/>
@@ -34,23 +32,9 @@
   <!-- Offset distance from the bottom border to the center of the wheel -->
   <xacro:property name="caster_z_offset" value="0.008"/>
-  <xacro:property name="caster_pos_x_joint" value="${(base_len/2) - caster_x_offset}"/>
-  <xacro:property name="caster_pos_y_joint" value="${(base_width/2) - caster_y_offset - (caster_height/2)}"/>
+  <xacro:property name="caster_pos_x_joint" value="${(base_props['base']['length']/2) - caster_x_offset}"/>
+  <xacro:property name="caster_pos_y_joint"
+    value="${(base_props['base']['width']/2) - caster_y_offset - (base_props['base']['height']/2)}"/>
   <xacro:property name="caster_pos_z_joint" value="${caster_z_offset}"/>
-  <!--Base link-->
-  <!-- <link name="base_link">
-    <xacro:box_inertia m="10" x="${base_len}" y="0.01" z="${base_width}" />
-    <visual>
-      <origin xyz="0 0 0" rpy="${PI/2} 0 -${PI/2}" />
-      <geometry>
-        <mesh filename="package://quimera_robot_description/meshes/quimera_struct.dae" />
-      </geometry>
-      <material name="white" />
-    </visual>
-    <collision>
-      <geometry>
-        <box size="${base_len} ${base_width} 0.01"/>
-      </geometry>
-    </collision>
-  </link> -->
+  <!-- Base link -->
   <xacro:base base_prop="${base_props}" mesh="${base_props['base']['mesh']}" >
     <origin xyz="0 0 0" rpy="${PI/2} 0 -${PI/2}" />

Commit message: Change base parameters name for the size in each axis.

File: urdf/common_macro.xacro (robot description, xacro)
@@ -47,7 +47,7 @@
     <link name="base_link">
     <xacro:box_inertia m="${base_prop['base']['mass']}"
-                       x="${base_prop['base']['length']}"
-                       y="${base_prop['base']['width']}"
-                       z="${base_prop['base']['height']}">
+                       x="${base_prop['base']['x_size']}"
+                       y="${base_prop['base']['y_size']}"
+                       z="${base_prop['base']['z_size']}">
     </xacro:box_inertia>
     <xacro:if value="${mesh != '' }" >
@@ -64,5 +64,5 @@
         <xacro:insert_block name="origin" />
         <geometry>
-          <box size="${base_prop['base']['length']} ${base_prop['base']['width']} ${base_prop['base']['height']}"/>
+          <box size="${base_prop['base']['x_size']} ${base_prop['base']['y_size']} ${base_prop['base']['z_size']}"/>
         </geometry>
         <material name="white" />
@@ -71,5 +71,5 @@
     <collision>
       <geometry>
-        <box size="${base_prop['base']['length']} ${base_prop['base']['width']} ${base_prop['base']['height']}"/>
+        <box size="${base_prop['base']['x_size']} ${base_prop['base']['y_size']} ${base_prop['base']['z_size']}"/>
       </geometry>
     </collision>

File: urdf/quimera.urdf.xacro (robot description, xacro)
@@ -18,7 +18,7 @@
   <!-- Back Wheel joint position -->
   <xacro:property name="b_wheel_pos_x_joint"
-     value="${(base_props['base']['length']/2) - b_wheel_x_offset}"/>
+     value="${(base_props['base']['x_size']/2) - b_wheel_x_offset}"/>
   <xacro:property name="b_wheel_pos_y_joint"
-    value="${(base_props['base']['width']/2) - b_wheel_y_offset - (wheel_props['wheel']['length']/2)}"/>
+    value="${(base_props['base']['y_size']/2) - b_wheel_y_offset - (wheel_props['wheel']['length']/2)}"/>
   <xacro:property name="b_wheel_pos_z_joint" value="${b_wheel_z_offset}"/>
   <!-- ######################################## -->
@@ -31,18 +31,21 @@
   <xacro:property name="f_wheel_z_offset" value="0.008"/>
   <!-- Front Wheel joint position -->
-  <xacro:property name="f_wheel_pos_x_joint" value="${(base_props['base']['length']/2) - f_wheel_x_offset}"/>
+  <xacro:property name="f_wheel_pos_x_joint" value="${(base_props['base']['x_size']/2) - f_wheel_x_offset}"/>
   <xacro:property name="f_wheel_pos_y_joint"
-    value="${(base_props['base']['width']/2) - f_wheel_y_offset - (front_wheel_props['wheel']['length']/2)}"/>
+    value="${(base_props['base']['y_size']/2) - f_wheel_y_offset - (front_wheel_props['wheel']['length']/2)}"/>
   <xacro:property name="f_wheel_pos_z_joint" value="${f_wheel_z_offset}"/>
   <!-- ######################################## -->
+  <!-- <xacro:macro name="get_parameters" params="yaml_name prefix">
+    <xacro:property name="yaml" value="$(find quimera_robot_description)/config/${yaml_name}.yaml" />
+    <xacro:property name="${prefix}_props" value="${load_yaml(yaml)}" scope="global"/>
+  </xacro:macro> -->
+  <!-- <xacro:get_parameters yaml_name="back_wheel" prefix="front"/> -->
+  <!-- <xacro:property name="test_props" value="${props}"/> -->
+  <!-- <xacro:get_parameters yaml_name="front_wheel"/>
+  <xacro:property name="front_props" value="${props}"/> -->
   <!-- Base link -->
   <xacro:base base_prop="${base_props}" mesh="${base_props['base']['mesh']}" >
     <origin xyz="0 0 0" rpy="${PI/2} 0 -${PI/2}" />
   </xacro:base>
-<!--
-  <xacro:macro name="test" params="x">
-    <xacro:property name="posi_x" value="0.008 | ${x}"/>
-  </xacro:macro>
-  <xacro:test x="2"/> -->
   <!-- Back Wheel -->
   <xacro:wheel prefix="back_right" reflect="-1"

Commit message: Change package name from quimera to mobile_robot_description.

File: urdf/common_macro.xacro (robot description, xacro)
@@ -11,5 +11,5 @@
         <origin xyz="0.0 0 0" rpy="${pi/2} 0 0"/>
          <geometry>
-        <mesh filename="package://quimera_robot_description/meshes/${mesh}.dae" />
+        <mesh filename="package://mobile_robot_description/meshes/${mesh}.dae" />
         </geometry>
       </visual>
@@ -55,5 +55,5 @@
         <xacro:insert_block name="origin" />
         <geometry>
-          <mesh filename="package://quimera_robot_description/meshes/${mesh}.dae" />
+          <mesh filename="package://mobile_robot_description/meshes/${mesh}.dae" />
         </geometry>
         <material name="white" />

File: urdf/quimera.urdf.xacro (robot description, xacro)
@@ -1,10 +1,10 @@
 <?xml version="1.0"?>
 <robot xmlns:xacro="http://www.ros.org/wiki/xacro" name="mobile_robot">
-  <xacro:include filename="$(find quimera_robot_description)/urdf/common_macro.xacro" />
-  <xacro:property name="back_wheel_yaml" value="$(find quimera_robot_description)/config/back_wheel.yaml" />
+  <xacro:include filename="$(find mobile_robot_description)/urdf/common_macro.xacro" />
+  <xacro:property name="back_wheel_yaml" value="$(find mobile_robot_description)/config/back_wheel.yaml" />
   <xacro:property name="wheel_props" value="${load_yaml(back_wheel_yaml)}"/>
-  <xacro:property name="front_wheel_yaml" value="$(find quimera_robot_description)/config/front_wheel.yaml" />
+  <xacro:property name="front_wheel_yaml" value="$(find mobile_robot_description)/config/front_wheel.yaml" />
   <xacro:property name="front_wheel_props" value="${load_yaml(front_wheel_yaml)}"/>
-  <xacro:property name="base_yaml" value="$(find quimera_robot_description)/config/base.yaml" />
+  <xacro:property name="base_yaml" value="$(find mobile_robot_description)/config/base.yaml" />
   <xacro:property name="base_props" value="${load_yaml(base_yaml)}"/>
   <xacro:property name="PI" value="3.14"/>
