Commit message: Remove unused lines and PI definition.

File: urdf/mobile_robot.urdf.xacro (robot description, xacro)
@@ -8,14 +8,7 @@
   <xacro:property name="base_yaml" value="$(find mobile_robot_description)/config/base.yaml" />
   <xacro:property name="base_props" value="${load_yaml(base_yaml)}"/>
-  <xacro:property name="PI" value="3.14"/>
-  <!-- <xacro:macro name="get_parameters" params="yaml_name prefix">
-    <xacro:property name="yaml" value="$(find quimera_robot_description)/config/${yaml_name}.yaml" />
-    <xacro:property name="${prefix}_props" value="${load_yaml(yaml)}" scope="global"/>
-  </xacro:macro> -->
-  <!-- <xacro:get_parameters yaml_name="back_wheel" prefix="front"/> -->
-  <!-- <xacro:property name="test_props" value="${props}"/> -->
   <!-- Base link -->
   <xacro:base base_prop="${base_props}" mesh="${base_props['base']['mesh']}" >
-    <origin xyz="0 0 0" rpy="${PI/2} 0 -${PI/2}" />
+    <origin xyz="0 0 0" rpy="${pi/2} 0 -${pi/2}" />
   </xacro:base>
   <!-- Back Wheels -->

Commit message: Add generic model.

File: urdf/mobile_robot.urdf.xacro (robot description, xacro)
@@ -5,5 +5,5 @@
   <!-- <xacro:set_package_name /> -->
   <xacro:property name="back_wheel_yaml" value="$(find ${package_name})/config/back_wheel.yaml" />
-  <xacro:property name="wheel_props" value="${load_yaml(back_wheel_yaml)}"/>
+  <xacro:property name="back_wheel_props" value="${load_yaml(back_wheel_yaml)}"/>
   <xacro:property name="front_wheel_yaml" value="$(find ${package_name})/config/front_wheel.yaml" />
   <xacro:property name="front_wheel_props" value="${load_yaml(front_wheel_yaml)}"/>
@@ -12,16 +12,16 @@
   <!-- Base link -->
   <xacro:base base_prop="${base_props}" mesh="${base_props['base']['mesh']}" >
-    <origin xyz="0 0 0" rpy="${pi/2} 0 -${pi/2}" />
+    <origin xyz="0 0 0" rpy="0 0 0" />
   </xacro:base>
   <!-- Back Wheels -->
   <xacro:wheel prefix="back_right" reflect="-1"
-                      wheel_props="${wheel_props}"
+                      wheel_props="${back_wheel_props}"
                       base_props="${base_props}"
-                      mesh="${wheel_props['wheel']['mesh']}">
+                      mesh="${back_wheel_props['wheel']['mesh']}">
   </xacro:wheel>
   <xacro:wheel prefix="back_left" reflect="1"
-                      wheel_props="${wheel_props}"
+                      wheel_props="${back_wheel_props}"
                       base_props="${base_props}"
-                      mesh="${wheel_props['wheel']['mesh']}">
+                      mesh="${back_wheel_props['wheel']['mesh']}">
   </xacro:wheel>
   <!-- Front Wheels -->
