Commit message: improve wheel property name.

File: urdf/quimera_robot.urdf.xacro (robot description, xacro)
@@ -6,5 +6,5 @@
   <!-- <xacro:set_package_name /> -->
   <xacro:property name="back_wheel_yaml" value="$(find ${package_name})/config/${robot_name}/back_wheel.yaml" />
-  <xacro:property name="wheel_props" value="${load_yaml(back_wheel_yaml)}"/>
+  <xacro:property name="back_wheel_props" value="${load_yaml(back_wheel_yaml)}"/>
   <xacro:property name="front_wheel_yaml" value="$(find ${package_name})/config/${robot_name}/front_wheel.yaml" />
   <xacro:property name="front_wheel_props" value="${load_yaml(front_wheel_yaml)}"/>
@@ -17,12 +17,12 @@
   <!-- Back Wheels -->
   <xacro:wheel prefix="back_right" reflect="-1"
-                      wheel_props="${wheel_props}"
+                      wheel_props="${back_wheel_props}"
                       base_props="${base_props}"
-                      mesh="${wheel_props['wheel']['mesh']}">
+                      mesh="${back_wheel_props['wheel']['mesh']}">
   </xacro:wheel>
   <xacro:wheel prefix="back_left" reflect="1"
-                      wheel_props="${wheel_props}"
+                      wheel_props="${back_wheel_props}"
                       base_props="${base_props}"
-                      mesh="${wheel_props['wheel']['mesh']}">
+                      mesh="${back_wheel_props['wheel']['mesh']}">
   </xacro:wheel>
   <!-- Front Wheels -->

Commit message: add hokuyo and adjust quimera_robot folder name.

File: urdf/quimera_robot.urdf.xacro (robot description, xacro)
@@ -2,6 +2,7 @@
 <robot xmlns:xacro="http://www.ros.org/wiki/xacro" name="quimera_robot">
   <xacro:property name="package_name" value="mobile_robot_description"/>
-  <xacro:property name="robot_name" value="quimera"/>
+  <xacro:property name="robot_name" value="quimera_robot"/>
   <xacro:include filename="$(find ${package_name})/urdf/include/common_macros.urdf.xacro" />
+  <xacro:include filename="$(find ${package_name})/urdf/include/common_sensors.xacro" />
   <xacro:include filename="$(find ${package_name})/urdf/quimera_robot.gazebo.xacro" />
   <xacro:property name="back_wheel_yaml" value="$(find ${package_name})/config/${robot_name}/back_wheel.yaml" />
@@ -35,3 +36,7 @@
                       base_props="${base_props}">
   </xacro:wheel>
+  <!-- Sensors -->
+  <xacro:hokuyo_sensor parent_link="base_link" >
+    <origin xyz="-0.02 0 ${base_props['base']['z_size'] + 0.05}" rpy="0 0 0" />
+  </xacro:hokuyo_sensor>
 </robot>
