Commit message: move diffbot config files to its own folder

File: urdf/diffbot.urdf.xacro (robot description, xacro)
@@ -2,11 +2,12 @@
 <robot xmlns:xacro="http://www.ros.org/wiki/xacro" name="mobile_robot">
   <xacro:property name="package_name" value="mobile_robot_description"/>
+  <xacro:property name="robot_name" value="diffbot"/>
   <xacro:include filename="$(find ${package_name})/urdf/include/common_macros.urdf.xacro" />
   <!-- <xacro:set_package_name /> -->
-  <xacro:property name="caster_wheel_yaml" value="$(find ${package_name})/config/caster_wheel.yaml" />
+  <xacro:property name="caster_wheel_yaml" value="$(find ${package_name})/config/${robot_name}/caster_wheel.yaml" />
   <xacro:property name="caster_wheel_props" value="${load_yaml(caster_wheel_yaml)}"/>
-  <xacro:property name="front_wheel_yaml" value="$(find ${package_name})/config/front_wheel.yaml" />
+  <xacro:property name="front_wheel_yaml" value="$(find ${package_name})/config/${robot_name}/front_wheel.yaml" />
   <xacro:property name="front_wheel_props" value="${load_yaml(front_wheel_yaml)}"/>
-  <xacro:property name="base_yaml" value="$(find ${package_name})/config/base.yaml" />
+  <xacro:property name="base_yaml" value="$(find ${package_name})/config/${robot_name}/base.yaml" />
   <xacro:property name="base_props" value="${load_yaml(base_yaml)}"/>
   <!-- Base link -->

Commit message: use new motor macros for diffbot

File: urdf/diffbot.urdf.xacro (robot description, xacro)
@@ -1,5 +1,5 @@
 <?xml version="1.0"?>
-<robot xmlns:xacro="http://www.ros.org/wiki/xacro" name="mobile_robot">
-  <xacro:property name="package_name" value="mobile_robot_description"/>
+<robot xmlns:xacro="http://www.ros.org/wiki/xacro" name="diffbot">
+  <xacro:property name="package_name" value="diffbot_description"/>
   <xacro:property name="robot_name" value="diffbot"/>
   <xacro:include filename="$(find ${package_name})/urdf/include/common_macros.urdf.xacro" />
@@ -9,4 +9,6 @@
   <xacro:property name="front_wheel_yaml" value="$(find ${package_name})/config/${robot_name}/front_wheel.yaml" />
   <xacro:property name="front_wheel_props" value="${load_yaml(front_wheel_yaml)}"/>
+  <xacro:property name="motor_yaml" value="$(find ${package_name})/config/${robot_name}/motor.yaml" />
+  <xacro:property name="motor_props" value="${load_yaml(motor_yaml)}"/>
   <xacro:property name="base_yaml" value="$(find ${package_name})/config/${robot_name}/base.yaml" />
   <xacro:property name="base_props" value="${load_yaml(base_yaml)}"/>
@@ -30,4 +32,15 @@
                       mesh="${front_wheel_props['wheel']['mesh']}">
   </xacro:wheel>
+  <!-- Motors -->
+  <xacro:motor prefix="right" reflect="-1"
+                      motor_props="${motor_props}"
+                      base_props="${base_props}"
+                      mesh="${motor_props['mesh']}">
+  </xacro:motor>
+  <xacro:motor prefix="left" reflect="1"
+                      motor_props="${motor_props}"
+                      base_props="${base_props}"
+                      mesh="${motor_props['mesh']}">
+  </xacro:motor>
   <!-- <xacro:include filename="$(find mobile_description)/urdf/mobile_robot_gazebo_plugins.xacro"/>  -->
 </robot>
