Commit message: WIP: add caster_wheel macro

File: urdf/include/common_macros.urdf.xacro (robot description, xacro)
@@ -41,4 +41,71 @@
       <origin xyz="${pos_x_joint} ${reflect* pos_y_joint} ${pos_z_joint}" rpy="0 0 0"/>
     </joint>
+  </xacro:macro>
+<!-- Caster wheel link & joint macro -->
+  <xacro:macro name="caster_wheel" params="locationprefix locationright wheel_base_dx
+    flipY:=${1}">
+    <!-- caster hub -->
+    <joint name="${locationprefix}_caster_rotation_joint" type="continuous">
+      <origin xyz="${wheel_base_dx} ${-caster_wheel_base_dy * locationright} ${caster_wheel_base_dz}" rpy="0 0 0" />
+      <parent link="base_link" />
+      <child link="${locationprefix}_caster_rotation_link" />
+      <axis xyz="0 0 1" />
+      <dynamics damping="0.01" friction="0.0"/>
+    </joint>
+    <link name="${locationprefix}_caster_rotation_link">
+      <inertial>
+        <origin xyz="0 0 ${-caster_base_size/2.0}" rpy="0 0 0" />
+        <mass value="${caster_base_mass}" />
+        <xacro:box_inertia  m="${caster_base_mass}" l="${caster_base_size}" w="${caster_base_size}" h="${caster_base_size}" />
+      </inertial>
+      <visual>
+        <origin xyz="0 0 ${-caster_base_size/2.0}" rpy="0 0 0" />
+        <geometry>
+          <!--mesh filename="package://mobile_robot_description/meshes/visual/caster_wheel_base.stl" /-->
+          <box size="${caster_base_size} ${caster_base_size} ${caster_base_size}" />
+        </geometry>
+        <xacro:insert_block name="material_silver" />
+      </visual>
+      <collision>
+        <origin xyz="0 0 ${-caster_base_size/2.0}" rpy="0 0 0" />
+        <geometry>
+          <!--mesh filename="package://mobile_robot_description/meshes/collision/caster_wheel_base.stl" /-->
+          <box size="${caster_base_size} ${caster_base_size} ${caster_base_size}" />
+        </geometry>
+      </collision>
+    </link>
+    <gazebo reference="${locationprefix}_caster_rotation_link">
+      <material>Gazebo/Grey</material>
+    </gazebo>
+    <!-- caster wheel -->
+    <joint name="${locationprefix}_caster_wheel_joint" type="continuous">
+      <origin xyz="${caster_wheel_dx} ${-caster_wheel_dy * locationright} ${caster_wheel_dz}" rpy="0 0 0" />
+      <parent link="${locationprefix}_caster_rotation_link" />
+      <child link="${locationprefix}_caster_wheel_link" />
+      <axis xyz="0 1 0" />
+    </joint>
+    <link name="${locationprefix}_caster_wheel_link">
+      <xacro:cylinder_inertial mass="${caster_wheel_mass}" radius="${caster_wheel_radius}" length="${caster_wheel_width}">
+        <origin xyz="0 0 0" rpy="${pi/2} 0 0" />
+      </xacro:cylinder_inertial>
+      <visual>
+        <origin xyz="0 0 0" rpy="${flipY*pi/2} 0 0" />
+        <geometry>
+          <!--mesh filename="package://mobile_robot_description/meshes/visual/wheel.stl" -->
+          <cylinder length="${caster_wheel_width}" radius="${caster_wheel_radius}" />
+        </geometry>
+        <xacro:insert_block name="material_dark_grey" />
+      </visual>
+      <collision>
+        <origin xyz="0 0 0" rpy="${flipY*pi/2} 0 0" />
+        <geometry>
+          <!--mesh filename="package://mobile_robot_description/meshes/visual/wheel.stl" -->
+          <cylinder length="${caster_wheel_width}" radius="${caster_wheel_radius}" />
+        </geometry>
+      </collision>
+    </link>
+    <gazebo reference="${locationprefix}_caster_wheel_link">
+        <material>Gazebo/DarkGrey</material>
+    </gazebo>
   </xacro:macro>
 <!--Base macro-->

File: urdf/mobile_robot.urdf.xacro (robot description, xacro)
@@ -1,5 +1,5 @@
 <?xml version="1.0"?>
 <robot xmlns:xacro="http://www.ros.org/wiki/xacro" name="mobile_robot">
-  <xacro:include filename="$(find mobile_robot_description)/urdf/common_macro.xacro" />
+  <xacro:include filename="$(find mobile_robot_description)/urdf/include/common_macros.urdf.xacro" />
   <xacro:property name="back_wheel_yaml" value="$(find mobile_robot_description)/config/back_wheel.yaml" />
   <xacro:property name="wheel_props" value="${load_yaml(back_wheel_yaml)}"/>

Commit message: Add joint position calculation to the xacro:wheel.

File: urdf/include/common_macros.urdf.xacro (robot description, xacro)
@@ -1,9 +1,12 @@
 <?xml version="1.0"?>
 <robot xmlns:xacro="http://www.ros.org/wiki/xacro">
-<!--Wheel link1 & joint macro-->
+<!--Wheel link & joint macro-->
   <xacro:macro name="wheel"
-               params="prefix reflect wheel_prop
-                       pos_x_joint pos_y_joint pos_z_joint mesh:=''">
-    <xacro:property name="radius" value="${wheel_props['wheel']['radius']}"/>
+               params="prefix reflect wheel_props base_props mesh:=''">
+  <xacro:property name="pos_x_joint"
+     value="${(base_props['base']['x_size']/2) - wheel_props['wheel']['x_offset']}"/>
+  <xacro:property name="pos_y_joint"
+    value="${(base_props['base']['y_size']/2) + wheel_props['wheel']['y_offset'] + (wheel_props['wheel']['length']/2)}"/>
+  <xacro:property name="pos_z_joint" value="${wheel_props['wheel']['z_offset']}"/>
     <link name="${prefix}_wheel">
     <xacro:if value="${mesh != '' }" >
@@ -19,5 +22,5 @@
         <origin xyz="0.0 0 0" rpy="${pi/2} 0 0"/>
          <geometry>
-         <cylinder radius="${wheel_prop['wheel']['radius']}" length="${wheel_prop['wheel']['length']}"/>
+         <cylinder radius="${wheel_props['wheel']['radius']}" length="${wheel_props['wheel']['length']}"/>
         </geometry>
         <material name="red"/>
@@ -27,10 +30,10 @@
         <origin xyz="0 0 0" rpy="${pi/2} 0 0"/>
         <geometry>
-          <cylinder radius="${wheel_prop['wheel']['radius']}" length="${wheel_prop['wheel']['length']}"/>
+          <cylinder radius="${wheel_props['wheel']['radius']}" length="${wheel_props['wheel']['length']}"/>
         </geometry>
       </collision>
-      <xacro:cylinder_inertia m="${wheel_prop['wheel']['mass']}"
-                              r="${wheel_prop['wheel']['radius']}"
-                              l="${wheel_prop['wheel']['length']}">
+      <xacro:cylinder_inertia m="${wheel_props['wheel']['mass']}"
+                              r="${wheel_props['wheel']['radius']}"
+                              l="${wheel_props['wheel']['length']}">
       </xacro:cylinder_inertia>
     </link>

File: urdf/mobile_robot.urdf.xacro (robot description, xacro)
@@ -9,18 +9,4 @@
   <xacro:property name="base_props" value="${load_yaml(base_yaml)}"/>
   <xacro:property name="PI" value="3.14"/>
-  <!-- Back Wheel joint position -->
-  <xacro:property name="b_wheel_pos_x_joint"
-     value="${(base_props['base']['x_size']/2) - wheel_props['wheel']['x_offset']}"/>
-  <xacro:property name="b_wheel_pos_y_joint"
-    value="${(base_props['base']['y_size']/2) + wheel_props['wheel']['y_offset'] + (wheel_props['wheel']['length']/2)}"/>
-  <xacro:property name="b_wheel_pos_z_joint" value="${wheel_props['wheel']['z_offset']}"/>
-  <!-- ######################################## -->
-  <!-- Front Wheel joint position -->
-  <xacro:property name="f_wheel_pos_x_joint"
-    value="${(base_props['base']['x_size']/2) - front_wheel_props['wheel']['x_offset']}"/>
-  <xacro:property name="f_wheel_pos_y_joint"
-    value="${(base_props['base']['y_size']/2) + front_wheel_props['wheel']['y_offset'] + (front_wheel_props['wheel']['length']/2)}"/>
-  <xacro:property name="f_wheel_pos_z_joint" value="${front_wheel_props['wheel']['z_offset']}"/>
-  <!-- ######################################## -->
   <!-- <xacro:macro name="get_parameters" params="yaml_name prefix">
     <xacro:property name="yaml" value="$(find quimera_robot_description)/config/${yaml_name}.yaml" />
@@ -35,29 +21,21 @@
   <!-- Back Wheels -->
   <xacro:wheel prefix="back_right" reflect="-1"
-                      wheel_prop="${wheel_props}"
-                      pos_x_joint="${b_wheel_pos_x_joint}"
-                      pos_y_joint="${b_wheel_pos_y_joint}"
-                      pos_z_joint="${b_wheel_pos_z_joint}"
+                      wheel_props="${wheel_props}"
+                      base_props="${base_props}"
                       mesh="${wheel_props['wheel']['mesh']}">
   </xacro:wheel>
   <xacro:wheel prefix="back_left" reflect="1"
-                      wheel_prop="${wheel_props}"
-                      pos_x_joint="${b_wheel_pos_x_joint}"
-                      pos_y_joint="${b_wheel_pos_y_joint}"
-                      pos_z_joint="${b_wheel_pos_z_joint}"
+                      wheel_props="${wheel_props}"
+                      base_props="${base_props}"
                       mesh="${wheel_props['wheel']['mesh']}">
   </xacro:wheel>
   <!-- Front Wheels -->
   <xacro:wheel prefix="front_right" reflect="-1"
-                      wheel_prop="${front_wheel_props}"
-                      pos_x_joint="${f_wheel_pos_x_joint}"
-                      pos_y_joint="${f_wheel_pos_y_joint}"
-                      pos_z_joint="${f_wheel_pos_z_joint}">
+                      wheel_props="${front_wheel_props}"
+                      base_props="${base_props}">
   </xacro:wheel>
   <xacro:wheel prefix="front_left" reflect="1"
-                      wheel_prop="${front_wheel_props}"
-                      pos_x_joint="${f_wheel_pos_x_joint}"
-                      pos_y_joint="${f_wheel_pos_y_joint}"
-                      pos_z_joint="${f_wheel_pos_z_joint}">
+                      wheel_props="${front_wheel_props}"
+                      base_props="${base_props}">
   </xacro:wheel>
   <!-- <xacro:include filename="$(find mobile_description)/urdf/mobile_robot_gazebo_plugins.xacro"/>  -->

Commit message: folder parametrization test.

File: urdf/include/common_macros.urdf.xacro (robot description, xacro)
@@ -3,5 +3,5 @@
 <!--Wheel link & joint macro-->
   <xacro:macro name="wheel"
-               params="prefix reflect wheel_props base_props mesh:=''">
+               params="prefix reflect wheel_props base_props mesh:='' ">
   <xacro:property name="pos_x_joint"
      value="${(base_props['base']['x_size']/2) - wheel_props['wheel']['x_offset']}"/>
@@ -114,5 +114,5 @@
 <!--Base macro-->
   <xacro:macro name="base"
-               params="base_prop mesh:='' *origin">
+               params="base_prop mesh:='' *origin name ">
     <link name="base_link">
     <xacro:box_inertia m="${base_prop['base']['mass']}"
@@ -125,5 +125,5 @@
         <xacro:insert_block name="origin" />
         <geometry>
-          <mesh filename="package://mobile_robot_description/meshes/${mesh}.dae" />
+          <mesh filename="package://${name}/meshes/${mesh}.dae" />
         </geometry>
         <material name="white" />

File: urdf/mobile_robot.urdf.xacro (robot description, xacro)
@@ -1,5 +1,6 @@
 <?xml version="1.0"?>
 <robot xmlns:xacro="http://www.ros.org/wiki/xacro" name="mobile_robot">
-  <xacro:include filename="$(find mobile_robot_description)/urdf/include/common_macros.urdf.xacro" />
+  <xacro:property name="folder_name" value="mobile_robot_description"/>
+  <xacro:include filename="$(find ${folder_name})/urdf/include/common_macros.urdf.xacro" />
   <xacro:property name="back_wheel_yaml" value="$(find mobile_robot_description)/config/back_wheel.yaml" />
   <xacro:property name="wheel_props" value="${load_yaml(back_wheel_yaml)}"/>
@@ -9,5 +10,5 @@
   <xacro:property name="base_props" value="${load_yaml(base_yaml)}"/>
   <!-- Base link -->
-  <xacro:base base_prop="${base_props}" mesh="${base_props['base']['mesh']}" >
+  <xacro:base base_prop="${base_props}" mesh="${base_props['base']['mesh']}" name="mobile_robot_description" >
     <origin xyz="0 0 0" rpy="${pi/2} 0 -${pi/2}" />
   </xacro:base>

Commit message: Make the package_name flexible.

File: urdf/include/common_macros.urdf.xacro (robot description, xacro)
@@ -1,4 +1,7 @@
 <?xml version="1.0"?>
 <robot xmlns:xacro="http://www.ros.org/wiki/xacro">
+<xacro:macro name="set_environment" params="package_name:='mobile_robot_description' ">
+  <xacro:property name="package_name" value="${package_name}" scope="global"/>
+</xacro:macro>
 <!--Wheel link & joint macro-->
   <xacro:macro name="wheel"
@@ -14,5 +17,5 @@
         <origin xyz="0.0 0 0" rpy="${pi/2} 0 0"/>
          <geometry>
-        <mesh filename="package://mobile_robot_description/meshes/${mesh}.dae" />
+        <mesh filename="package://${package_name}/meshes/${mesh}.dae" />
         </geometry>
       </visual>
@@ -114,5 +117,5 @@
 <!--Base macro-->
   <xacro:macro name="base"
-               params="base_prop mesh:='' *origin name ">
+               params="base_prop mesh:='' *origin ">
     <link name="base_link">
     <xacro:box_inertia m="${base_prop['base']['mass']}"
@@ -125,5 +128,6 @@
         <xacro:insert_block name="origin" />
         <geometry>
-          <mesh filename="package://${name}/meshes/${mesh}.dae" />
+          <!-- The folder path get a folder_name global parameter -->
+          <mesh filename="package://${package_name}/meshes/${mesh}.dae" />
         </geometry>
         <material name="white" />

File: urdf/mobile_robot.urdf.xacro (robot description, xacro)
@@ -1,14 +1,15 @@
 <?xml version="1.0"?>
 <robot xmlns:xacro="http://www.ros.org/wiki/xacro" name="mobile_robot">
-  <xacro:property name="folder_name" value="mobile_robot_description"/>
-  <xacro:include filename="$(find ${folder_name})/urdf/include/common_macros.urdf.xacro" />
-  <xacro:property name="back_wheel_yaml" value="$(find mobile_robot_description)/config/back_wheel.yaml" />
+  <xacro:property name="package_name" value="mobile_robot_description"/>
+  <xacro:include filename="$(find ${package_name})/urdf/include/common_macros.urdf.xacro" />
+  <!-- <xacro:set_package_name /> -->
+  <xacro:property name="back_wheel_yaml" value="$(find ${package_name})/config/back_wheel.yaml" />
   <xacro:property name="wheel_props" value="${load_yaml(back_wheel_yaml)}"/>
-  <xacro:property name="front_wheel_yaml" value="$(find mobile_robot_description)/config/front_wheel.yaml" />
+  <xacro:property name="front_wheel_yaml" value="$(find ${package_name})/config/front_wheel.yaml" />
   <xacro:property name="front_wheel_props" value="${load_yaml(front_wheel_yaml)}"/>
-  <xacro:property name="base_yaml" value="$(find mobile_robot_description)/config/base.yaml" />
+  <xacro:property name="base_yaml" value="$(find ${package_name})/config/base.yaml" />
   <xacro:property name="base_props" value="${load_yaml(base_yaml)}"/>
   <!-- Base link -->
-  <xacro:base base_prop="${base_props}" mesh="${base_props['base']['mesh']}" name="mobile_robot_description" >
+  <xacro:base base_prop="${base_props}" mesh="${base_props['base']['mesh']}" >
     <origin xyz="0 0 0" rpy="${pi/2} 0 -${pi/2}" />
   </xacro:base>
