Commit message: use robot_name property to unify yaml configs - avoid robot name in yaml

File: urdf/include/common_macros.urdf.xacro (robot description, xacro)
@@ -17,5 +17,5 @@
         <origin xyz="0.0 0 0" rpy="${pi/2} 0 ${pi/2.0*(reflect - 1)}"/>
          <geometry>
-        <mesh filename="package://${package_name}/meshes/${mesh}" />
+        <mesh filename="package://${package_name}/meshes/${robot_name}/${mesh}" />
         </geometry>
       </visual>
@@ -66,5 +66,5 @@
             <origin xyz="0 0 ${-wheel_props['base']['size']['z']/2.0}" rpy="0 0 0" />
             <geometry>
-                <mesh filename="package://${package_name}/meshes/${wheel_props['base']['mesh']}" />
+                <mesh filename="package://${package_name}/meshes/${robot_name}/${wheel_props['base']['mesh']}" />
             </geometry>
             <!-- xacro:insert_block name="material_silver" / TODO use this block? -->
@@ -113,5 +113,5 @@
           <origin xyz="0 0 ${-wheel_props['hub']['size']['z']/2.0}" rpy="0 0 0" />
           <geometry>
-            <mesh filename="package://${package_name}/meshes/${wheel_props['hub']['mesh']}" />
+            <mesh filename="package://${package_name}/meshes/${robot_name}/${wheel_props['hub']['mesh']}" />
           </geometry>
           <!-- xacro:insert_block name="material_silver" / TODO use this block? -->
@@ -157,5 +157,5 @@
           <origin xyz="0 0 0" rpy="0 0 0" />
           <geometry>
-            <mesh filename="package://${package_name}/meshes/${wheel_props['wheel']['mesh']}" />
+            <mesh filename="package://${package_name}/meshes/${robot_name}/${wheel_props['wheel']['mesh']}" />
           </geometry>
           <!-- TODO use this?: xacro:insert_block name="material_dark_grey" /-->
@@ -204,5 +204,5 @@
         <geometry>
           <!-- The folder path get a folder_name global parameter -->
-          <mesh filename="package://${package_name}/meshes/${mesh}" />
+          <mesh filename="package://${package_name}/meshes/${robot_name}/${mesh}" />
         </geometry>
         <material name="white" />

File: urdf/mobile_robot.urdf.xacro (robot description, xacro)
@@ -2,11 +2,12 @@
 <robot xmlns:xacro="http://www.ros.org/wiki/xacro" name="mobile_robot">
   <xacro:property name="package_name" value="mobile_robot_description"/>
+  <xacro:property name="robot_name" value="quimera"/>
   <xacro:include filename="$(find ${package_name})/urdf/include/common_macros.urdf.xacro" />
   <!-- <xacro:set_package_name /> -->
-  <xacro:property name="back_wheel_yaml" value="$(find ${package_name})/config/back_wheel.yaml" />
+  <xacro:property name="back_wheel_yaml" value="$(find ${package_name})/config/${robot_name}/back_wheel.yaml" />
   <xacro:property name="wheel_props" value="${load_yaml(back_wheel_yaml)}"/>
-  <xacro:property name="front_wheel_yaml" value="$(find ${package_name})/config/front_wheel.yaml" />
+  <xacro:property name="front_wheel_yaml" value="$(find ${package_name})/config/${robot_name}/front_wheel.yaml" />
   <xacro:property name="front_wheel_props" value="${load_yaml(front_wheel_yaml)}"/>
-  <xacro:property name="base_yaml" value="$(find ${package_name})/config/base.yaml" />
+  <xacro:property name="base_yaml" value="$(find ${package_name})/config/${robot_name}/base.yaml" />
   <xacro:property name="base_props" value="${load_yaml(base_yaml)}"/>
   <!-- Base link -->

Commit message: remove conflict.
Signed-off-by: pxalcantara <pxalcantara@gmail.com>

File: urdf/include/common_macros.urdf.xacro (robot description, xacro)
@@ -4,5 +4,7 @@
   <xacro:property name="package_name" value="${package_name}" scope="global"/>
 </xacro:macro>
-<!--Wheel link & joint macro-->
+<!--
+  Xacro to create a wheel link and the respective joint
+-->
   <xacro:macro name="wheel"
                params="prefix reflect wheel_props base_props mesh:='' ">
@@ -204,9 +206,5 @@
         <geometry>
           <!-- The folder path get a folder_name global parameter -->
-<<<<<<< HEAD
-          <mesh filename="package://${package_name}/meshes/${mesh}" />
-=======
           <mesh filename="package://${package_name}/meshes/${robot_name}/${mesh}" />
->>>>>>> 9360dda1a6d989eecddd3a32787117e0e6d87a18
         </geometry>
         <material name="white" />

Commit message: Add xacro comments documentation.
Signed-off-by: pxalcantara <pxalcantara@gmail.com>

File: urdf/include/common_macros.urdf.xacro (robot description, xacro)
@@ -4,6 +4,14 @@
   <xacro:property name="package_name" value="${package_name}" scope="global"/>
 </xacro:macro>
-<!--
-  Xacro to create a wheel link and the respective joint
+<!-- ===================== Wheel xacro =========================================
+  Xacro to create a wheel link and the respective joint. For more detail information and usage, see:
+    https://github.com/pxalcantara/mobile_robot_description/wiki/Wheel-xacro
+  params:
+  - prefix [string]: used to diferentiate the link and joint name;
+  - reflect [1/-1]: value to set the side of the wheel;
+  - wheel_props [dictionary]: wheel properties;
+  - base_props [dictionary]: base link properties;
+  - mesh [string]: file name of the wheel mesh;
+    - DEFAULT Value -> Empty string
 -->
   <xacro:macro name="wheel"
@@ -50,4 +58,5 @@
     </joint>
   </xacro:macro>
+<!-- ======================================================================= -->
 <!-- Caster wheel link & joint macro -->
   <!-- locationprefix locationright wheel_base_dx TODO remove -->
@@ -192,5 +201,11 @@
     </gazebo>
   </xacro:macro>
-<!--Base macro-->
+<!-- ===================== Base xacro ==========================================
+  Xacro to create the base link. For more detail information and usage, see:
+    https://github.com/pxalcantara/mobile_robot_description/wiki/Base-xacro
+  params:
+  - base_props [dictionary]: base link properties;
+  - origin [block]: origin, position and orientation of the link;
+-->
   <xacro:macro name="base"
                params="base_prop mesh:='' *origin ">
@@ -227,5 +242,14 @@
     </link>
   </xacro:macro>
-<!--Intertial macros-->
+<!-- ======================================================================= -->
+<!-- ======================= Intertial macros ===============================-->
+<!-- ===================== Cylinder intertia xacro =============================
+  Xacro with the intertial block of a cylinder. For more detail information and usage, see:
+    https://github.com/pxalcantara/mobile_robot_description/wiki/Inertia-xacro
+  params:
+  - m [float]: link mass;
+  - r [float]: cylinder radius;
+  - l [float]: cylinder lenght (height);
+-->
   <xacro:macro name="cylinder_inertia" params="m r l">
     <inertial>
@@ -235,4 +259,13 @@
     </inertial>
   </xacro:macro>
+<!-- ===================== Box intertia xacro ==================================
+  Xacro with the intertial block of a box. For more detail information and usage, see:
+    https://github.com/pxalcantara/mobile_robot_description/wiki/Inertia-xacro
+  params:
+  - m [float]: link mass;
+  - x [float]: link dimension on the X-axis;
+  - y [float]: link dimension on the Y-axis;
+  - z [float]: link dimension on the Z-axis;
+-->
  <xacro:macro name="box_inertia" params="m x y z">
     <inertial>
@@ -243,4 +276,11 @@
     </inertial>
   </xacro:macro>
+<!-- ===================== Sphere intertia xacro ===============================
+  Xacro with the intertial block of a sphere. For more detail information and usage, see:
+    https://github.com/pxalcantara/mobile_robot_description/wiki/Inertia-xacro
+  params:
+  - m [float]: link mass;
+  - r [float]: sphere radius;
+-->
   <xacro:macro name="sphere_inertia" params="m r">
     <inertial>
@@ -249,4 +289,10 @@
     </inertial>
   </xacro:macro>
+<!-- ===================== Default intertial xacro =============================
+  Xacro with a identity intertial block. For more detail information and usage, see:
+    https://github.com/pxalcantara/mobile_robot_description/wiki/Inertia-xacro
+  params:
+  - m [float]: link mass;
+-->
   <xacro:macro name="default_inertial" params="mass">
     <inertial>
@@ -255,5 +301,8 @@
     </inertial>
   </xacro:macro>
-<!--Color Properties-->
+<!-- ========================================================================-->
+<!-- ===================== Material ============================================
+  RVIZ material RGBA definition.
+-->
   <material name="blue">
     <color rgba="0 0 0.8 1"/>
@@ -274,8 +323,4 @@
     <color rgba="0.3 0.3 0.3 1"/>
   </material>
-  <!-- TODO use this?: xacro:property name="material_silver">
-    <material name="silver">
-      <color rgba="0.79 0.82 0.93 1" />
-    </material>
-  </xacro:property-->
+<!-- ========================================================================-->
 </robot>

Commit message: add mobile_robot config folder and files
Signed-off-by: pxalcantara <pxalcantara@gmail.com>

File: urdf/include/common_macros.urdf.xacro (robot description, xacro)
@@ -206,4 +206,6 @@
   params:
   - base_props [dictionary]: base link properties;
+  - mesh [string]: file name of the link mesh;
+    - DEFAULT Value -> Empty string
   - origin [block]: origin, position and orientation of the link;
 -->

File: urdf/mobile_robot.urdf.xacro (robot description, xacro)
@@ -2,8 +2,8 @@
 <robot xmlns:xacro="http://www.ros.org/wiki/xacro" name="mobile_robot">
   <xacro:property name="package_name" value="mobile_robot_description"/>
-  <xacro:property name="robot_name" value="quimera"/>
+  <xacro:property name="robot_name" value="mobile_robot"/>
   <xacro:include filename="$(find ${package_name})/urdf/include/common_macros.urdf.xacro" />
   <!-- <xacro:set_package_name /> -->
-  <xacro:property name="back_wheel_yaml" value="$(find ${package_name})/config/back_wheel.yaml" />
+  <xacro:property name="back_wheel_yaml" value="$(find ${package_name})/config/${robot_name}/back_wheel.yaml" />
   <xacro:property name="back_wheel_props" value="${load_yaml(back_wheel_yaml)}"/>
   <xacro:property name="front_wheel_yaml" value="$(find ${package_name})/config/${robot_name}/front_wheel.yaml" />
@@ -12,5 +12,5 @@
   <xacro:property name="base_props" value="${load_yaml(base_yaml)}"/>
   <!-- Base link -->
-  <xacro:base base_prop="${base_props}" mesh="${base_props['base']['mesh']}" >
+  <xacro:base base_prop="${base_props}" >
     <origin xyz="0 0 0" rpy="0 0 0" />
   </xacro:base>

Commit message: Update quimera base link and position.

File: urdf/include/common_macros.urdf.xacro (robot description, xacro)
@@ -238,4 +238,5 @@
     </xacro:if>
     <collision>
+      <origin xyz="0 0 0.09" rpy="0 0 0"/>
       <geometry>
         <box size="${base_prop['base']['x_size']} ${base_prop['base']['y_size']} ${base_prop['base']['z_size']}"/>

File: urdf/quimera_robot.urdf.xacro (robot description, xacro)
@@ -4,4 +4,5 @@
   <xacro:property name="robot_name" value="quimera"/>
   <xacro:include filename="$(find ${package_name})/urdf/include/common_macros.urdf.xacro" />
+  <xacro:include filename="$(find ${package_name})/urdf/quimera_robot.gazebo.xacro" />
   <!-- <xacro:set_package_name /> -->
   <xacro:property name="back_wheel_yaml" value="$(find ${package_name})/config/${robot_name}/back_wheel.yaml" />
@@ -13,5 +14,5 @@
   <!-- Base link -->
   <xacro:base base_prop="${base_props}" mesh="${base_props['base']['mesh']}" >
-    <origin xyz="0 0 0" rpy="${pi/2} 0 -${pi/2}" />
+    <origin xyz="0 0 0" rpy="0 0 ${pi/2}" />
   </xacro:base>
   <!-- Back Wheels -->
@@ -35,4 +36,3 @@
                       base_props="${base_props}">
   </xacro:wheel>
-  <!-- <xacro:include filename="$(find mobile_description)/urdf/mobile_robot_gazebo_plugins.xacro"/>  -->
 </robot>

Commit message: add transmission to the wheels:xacro.

File: urdf/include/common_macros.urdf.xacro (robot description, xacro)
@@ -57,4 +57,14 @@
       <origin xyz="${pos_x_joint} ${reflect* pos_y_joint} ${pos_z_joint}" rpy="0 0 0"/>
     </joint>
+    <transmission name="${prefix}_wheel_transmission">
+      <type>transmission_interface/SimpleTransmission</type>
+      <joint name="${prefix}_wheel_joint">
+        <hardwareInterface>hardware_interface/VelocityJointInterface</hardwareInterface>
+      </joint>
+      <actuator name="${prefix}_motor">
+        <hardwareInterface>hardware_interface/VelocityJointInterface</hardwareInterface>
+        <mechanicalReduction>1</mechanicalReduction>
+      </actuator>
+    </transmission>
   </xacro:macro>
 <!-- ======================================================================= -->

Commit message: remove whitespace; rename material_dark_grey to dark_grey

File: urdf/include/common_macros.urdf.xacro (robot description, xacro)
@@ -26,7 +26,8 @@
       <visual>
         <origin xyz="0.0 0 0" rpy="${pi/2} 0 ${pi/2.0*(reflect - 1)}"/>
-         <geometry>
-        <mesh filename="package://${package_name}/meshes/${robot_name}/${mesh}" />
-        </geometry>
+        <geometry>
+          <mesh filename="package://${package_name}/meshes/${robot_name}/${mesh}" />
+        </geometry>
+        <material name="dark_grey"/>
       </visual>
     </xacro:if>
@@ -181,5 +182,5 @@
           </geometry>
           <!-- TODO use this?: xacro:insert_block name="material_dark_grey" /-->
-          <material name="material_dark_grey"/>
+          <material name="dark_grey"/>
         </visual>
       </xacro:if>
@@ -333,5 +334,5 @@
     <color rgba="0.79 0.82 0.93 1"/>
   </material>
-  <material name="material_dark_grey">
+  <material name="dark_grey">
     <color rgba="0.3 0.3 0.3 1"/>
   </material>

Commit message: add motor xacro macro

File: urdf/include/common_macros.urdf.xacro (robot description, xacro)
@@ -212,4 +212,66 @@
     </gazebo>
   </xacro:macro>
+<!-- ===================== Motor xacro =========================================
+  Xacro to create a motor link and the respective joint. For more detail information and usage, see:
+    https://github.com/pxalcantara/mobile_robot_description/wiki/Motor-xacro
+  params:
+  - prefix [string]: used to diferentiate the link and joint name;
+  - reflect [1/-1]: value to set the side of the motor;
+  - motor_props [dictionary]: motor properties;
+  - base_props [dictionary]: base link properties;
+  - mesh [string]: file name of the motor mesh;
+    - DEFAULT Value -> Empty string
+-->
+  <xacro:macro name="motor"
+               params="prefix reflect motor_props base_props mesh:='' ">
+  <xacro:property name="pos_x_joint"
+     value="${(base_props['base']['x_size']/2) - motor_props['x_offset']}"/>
+  <xacro:property name="pos_y_joint"
+    value="${(base_props['base']['y_size']/2) + motor_props['y_offset'] + (motor_props['y_size']/2)}"/>
+  <xacro:property name="pos_z_joint" value="${motor_props['z_offset']}"/>
+    <link name="${prefix}_motor">
+    <xacro:if value="${mesh != '' }" >
+      <visual>
+        <origin xyz="0.0 0.0 0.0" rpy="0.0 0 ${pi/2.0*(reflect - 1)}"/>
+        <geometry>
+          <mesh filename="package://${package_name}/meshes/${robot_name}/${mesh}" />
+        </geometry>
+        <material name="blue"/>
+      </visual>
+    </xacro:if>
+    <xacro:if value="${mesh == '' }" >
+      <visual>
+        <origin xyz="0.0 0 0" rpy="${pi/2} 0 0"/>
+         <geometry>
+          <box size="${motor_props['x_size']} ${motor_props['y_size']} ${motor_props['z_size']}"/>
+        </geometry>
+        <material name="red"/>
+      </visual>
+    </xacro:if>
+      <collision>
+        <origin xyz="0 0 0" rpy="${pi/2} 0 0"/>
+        <geometry>
+          <box size="${motor_props['x_size']} ${motor_props['y_size']} ${motor_props['z_size']}"/>
+        </geometry>
+      </collision>
+      <xacro:box_inertia m="${motor_props['mass']}"
+                         x="${motor_props['x_size']}"
+                         y="${motor_props['y_size']}"
+                         z="${motor_props['z_size']}">
+      </xacro:box_inertia>
+    </link>
+    <joint name="${prefix}_motor_joint" type="fixed">
+      <parent link="base_link"/>
+      <child link="${prefix}_motor"/>
+      <origin xyz="${pos_x_joint} ${reflect* pos_y_joint} ${pos_z_joint}" rpy="0 ${-pi/2.0*(reflect - 1)} 0"/>
+      <axis xyz="0 1 0" rpy="0 0 0" />
+      <!--origin xyz="${transX} ${reflect * (transY - wheel_width)} ${transZ}" rpy="${-pi/2.0*(reflect - 1)} 0 0" /-->
+      <!--axis xyz="0 1 0" rpy="0 0 ${pi/2.0*(reflect - 1)}" /-->
+    </joint>
+    <!--gazebo reference="${fb}_${lr}_motor">
+      <material>Gazebo/SkyBlue</material>
+      <turnGravityOff>false</turnGravityOff>
+    </gazebo-->
+  </xacro:macro>
 <!-- ===================== Base xacro ==========================================
   Xacro to create the base link. For more detail information and usage, see:

Commit message: Update common_macros.urdf.xacro; fix inertia/collision
- add origin to box_inertia and cylinder_inertia macro (used for e.g.
  castor wheel)
- fix base link collision (removed offset error)
- fix wheel inertia (rotate by pi/2)
- add base footprint link and joint (common for mobile base robots)

File: urdf/include/common_macros.urdf.xacro (robot description, xacro)
@@ -49,5 +49,7 @@
       <xacro:cylinder_inertia m="${wheel_props['wheel']['mass']}"
                               r="${wheel_props['wheel']['radius']}"
-                              l="${wheel_props['wheel']['length']}">
+                              l="${wheel_props['wheel']['length']}"
+                              o_xyz="0.0 0.0 0.0"
+                              o_rpy="${pi/2.0} 0.0 0.0" >
       </xacro:cylinder_inertia>
     </link>
@@ -76,12 +78,10 @@
     <!-- caster base (fixed) -->
     <link name="${prefix}_caster_base_link">
-      <inertial>
-        <origin xyz="0 0 ${-wheel_props['base']['size']['z']/2.0}" rpy="0 0 0" />
-        <mass value="${wheel_props['base']['mass']}" />
-        <xacro:box_inertia  m="${wheel_props['base']['mass']}"
-                            x="${wheel_props['base']['size']['x']}"
-                            y="${wheel_props['base']['size']['y']}"
-                            z="${wheel_props['base']['size']['z']}" />
-      </inertial>
+      <xacro:box_inertia  m="${wheel_props['base']['mass']}"
+                          x="${wheel_props['base']['size']['x']}"
+                          y="${wheel_props['base']['size']['y']}"
+                          z="${wheel_props['base']['size']['z']}"
+                          o_xyz="0.0 0.0 ${-wheel_props['base']['size']['z']/2.0}"
+                          o_rpy="0.0 0.0 0.0" />
       <xacro:if value="${wheel_props['base']['mass'] != '' }" >
         <visual>
@@ -123,12 +123,10 @@
     <!-- caster hub -->
     <link name="${prefix}_caster_rotation_link">
-      <inertial>
-        <origin xyz="0 0 ${-wheel_props['hub']['size']['z']/2.0}" rpy="0 0 0" />
-        <mass value="${wheel_props['hub']['mass']}" />
-        <xacro:box_inertia  m="${wheel_props['hub']['mass']}"
-                            x="${wheel_props['hub']['size']['x']}"
-                            y="${wheel_props['hub']['size']['y']}"
-                            z="${wheel_props['hub']['size']['z']}" />
-      </inertial>
+      <xacro:box_inertia  m="${wheel_props['hub']['mass']}"
+                          x="${wheel_props['hub']['size']['x']}"
+                          y="${wheel_props['hub']['size']['y']}"
+                          z="${wheel_props['hub']['size']['z']}"
+                          o_xyz="0.0 0.0 ${-wheel_props['hub']['size']['z']/2.0}"
+                          o_rpy="0.0 0.0 0.0" />
       <xacro:if value="${wheel_props['hub']['mesh'] != '' }" >
         <visual>
@@ -171,6 +169,6 @@
     <link name="${prefix}_caster_wheel_link">
       <xacro:cylinder_inertia m="${wheel_props['wheel']['mass']}"
-                            r="${wheel_props['wheel']['radius']}"
-                            l="${wheel_props['wheel']['length']}">
+                              r="${wheel_props['wheel']['radius']}"
+                              l="${wheel_props['wheel']['length']}">
         <!-- TODO unused block error?: origin xyz="0 0 0" rpy="${pi/2} 0 0" /-->
       </xacro:cylinder_inertia>
@@ -311,5 +309,5 @@
     </xacro:if>
     <collision>
-      <origin xyz="0 0 0.09" rpy="0 0 0"/>
+      <origin xyz="0.0 0.0 0.0" rpy="0.0 0.0 0.0"/>
       <geometry>
         <box size="${base_prop['base']['x_size']} ${base_prop['base']['y_size']} ${base_prop['base']['z_size']}"/>
@@ -317,4 +315,27 @@
     </collision>
     </link>
+  </xacro:macro>
+<!-- ===================== Footprint xacro ==========================================
+  Xacro to create the base link. For more detail information and usage, see:
+    https://github.com/pxalcantara/mobile_robot_description/wiki/Base-xacro
+  params:
+  - base_props [dictionary]: base link properties;
+  - mesh [string]: file name of the link mesh;
+    - DEFAULT Value -> Empty string
+  - origin [block]: origin, position and orientation of the link;
+-->
+  <xacro:macro name="footprint"
+               params="wheel_props">
+    <!-- Base-Footprint -->
+    <!-- base_footprint is a fictitious link(frame) that is on the ground right below base_link origin -->
+    <link name="base_footprint" />
+    <!-- Joint to connect base_footprint with base_link -->
+    <joint name="base_footprint_joint" type="fixed">
+      <parent link="base_footprint"/>
+      <child link="base_link" />
+      <!-- origin xyz="0 0 ${wheel_radius - base_z_origin_to_wheel_origin}" rpy="0 0 0" /-->
+      <!-- origin xyz="0 0 ${wheel_props['wheel']['radius'] - wheel_props['wheel']['z_offset'] + 0.1}" rpy="0 0 0" /-->
+      <origin xyz="0 0 0" rpy="0 0 0" />
+    </joint>
   </xacro:macro>
 <!-- ======================================================================= -->
@@ -328,9 +349,10 @@
   - l [float]: cylinder lenght (height);
 -->
-  <xacro:macro name="cylinder_inertia" params="m r l">
+  <xacro:macro name="cylinder_inertia" params="m r l o_xyz:='0.0 0.0 0.0' o_rpy:='0.0 0.0 0.0'">
     <inertial>
       <mass value="${m}"/>
       <inertia ixx="${m*(3*r*r+l*l)/12}" ixy = "0" ixz = "0"
                iyy="${m*(3*r*r+l*l)/12}" iyz = "0" izz="${m*r*r/2}"/>
+      <origin xyz="${o_xyz}" rpy="${o_rpy}" />
     </inertial>
   </xacro:macro>
@@ -344,5 +366,5 @@
   - z [float]: link dimension on the Z-axis;
 -->
- <xacro:macro name="box_inertia" params="m x y z">
+ <xacro:macro name="box_inertia" params="m x y z o_xyz:='0.0 0.0 0.0' o_rpy:='0.0 0.0 0.0'">
     <inertial>
       <mass value="${m}"/>
@@ -350,4 +372,5 @@
                iyy="${m / 12.0 * (x*x + z*z)}" iyz="0.0"
                izz="${m / 12.0 * (x*x + y*y)}"/>
+      <origin xyz="${o_xyz}" rpy="${o_rpy}" />
     </inertial>
   </xacro:macro>
