Commit message: Add footprint link and hokuyo sensor

File: urdf/include/common_macros.urdf.xacro (robot description, xacro)
@@ -256,4 +256,22 @@
   </xacro:macro>
 <!-- ======================================================================= -->
+<!-- ===================== Footprint xacro ==========================================
+  Xacro to create the footprint link and creat a fixed joint with the base link.
+  params:
+  - wheel_props [dictionary]: wheel link properties;
+-->
+  <xacro:macro name="footprint"
+               params="wheel_props">
+    <!-- Base-Footprint -->
+    <!-- base_footprint is a fictitious link(frame) that is on the ground right below base_link origin -->
+    <link name="base_footprint" />
+    <!-- Joint to connect base_footprint with base_link -->
+    <joint name="base_footprint_joint" type="fixed">
+      <parent link="base_footprint"/>
+      <child link="base_link" />
+      <origin xyz="0 0 ${wheel_props['wheel']['radius'] - wheel_props['wheel']['z_offset']}" rpy="0 0 0" />
+    </joint>
+  </xacro:macro>
+<!-- ======================================================================= -->
 <!-- ======================= Intertial macros ===============================-->
 <!-- ===================== Cylinder intertia xacro =============================

File: urdf/quimera_robot.urdf.xacro (robot description, xacro)
@@ -6,4 +6,5 @@
   <xacro:include filename="$(find ${package_name})/urdf/include/common_sensors.xacro" />
   <xacro:include filename="$(find ${package_name})/urdf/quimera_robot.gazebo.xacro" />
+  <!-- <xacro:include filename="$(find hector_sensors_description)/urdf/generic_camera.urdf.xacro" /> -->
   <xacro:property name="back_wheel_yaml" value="$(find ${package_name})/config/${robot_name}/back_wheel.yaml" />
   <xacro:property name="back_wheel_props" value="${load_yaml(back_wheel_yaml)}"/>
@@ -12,4 +13,6 @@
   <xacro:property name="base_yaml" value="$(find ${package_name})/config/${robot_name}/base.yaml" />
   <xacro:property name="base_props" value="${load_yaml(base_yaml)}"/>
+  <!-- Footprint link -->
+  <xacro:footprint wheel_props="${back_wheel_props}" />
   <!-- Base link -->
   <xacro:base base_prop="${base_props}" mesh="${base_props['base']['mesh']}" >
@@ -40,3 +43,8 @@
     <origin xyz="-0.02 0 ${base_props['base']['z_size'] + 0.05}" rpy="0 0 0" />
   </xacro:hokuyo_sensor>
+  <!-- <xacro:generic_camera name="camera" parent="base_link" ros_topic="image_raw"
+                        cam_info_topic="camera_info" update_rate="30"
+                        res_x="800" res_y="800" image_format="R8G8B8" h_fov="1.4" >
+        <origin xyz="0 0 0" rpy="0 0 0" />
+  </xacro:generic_camera>                       -->
 </robot>

Commit message: adjust gazebo references

File: urdf/include/common_macros.urdf.xacro (robot description, xacro)
@@ -27,5 +27,5 @@
         <origin xyz="0.0 0 0" rpy="${pi/2} 0 ${pi/2.0*(reflect - 1)}"/>
          <geometry>
-        <mesh filename="package://${package_name}/meshes/${robot_name}/${mesh}" />
+        <mesh filename="file://$(find ${package_name})/meshes/${robot_name}/${mesh}" />
         </geometry>
       </visual>
@@ -57,5 +57,5 @@
       <origin xyz="${pos_x_joint} ${reflect* pos_y_joint} ${pos_z_joint}" rpy="0 0 0"/>
     </joint>
-    <transmission name="${prefix}_wheel_transmission">
+    <!-- <transmission name="${prefix}_wheel_transmission">
       <type>transmission_interface/SimpleTransmission</type>
       <joint name="${prefix}_wheel_joint">
@@ -66,5 +66,5 @@
         <mechanicalReduction>1</mechanicalReduction>
       </actuator>
-    </transmission>
+    </transmission> -->
   </xacro:macro>
 <!-- ======================================================================= -->
@@ -134,5 +134,5 @@
           <origin xyz="0 0 ${-wheel_props['hub']['size']['z']/2.0}" rpy="0 0 0" />
           <geometry>
-            <mesh filename="package://${package_name}/meshes/${robot_name}/${wheel_props['hub']['mesh']}" />
+            <mesh filename="file://${package_name}/meshes/${robot_name}/${wheel_props['hub']['mesh']}" />
           </geometry>
           <!-- xacro:insert_block name="material_silver" / TODO use this block? -->
@@ -233,5 +233,5 @@
         <geometry>
           <!-- The folder path get a folder_name global parameter -->
-          <mesh filename="package://${package_name}/meshes/${robot_name}/${mesh}" />
+          <mesh filename="file://$(find ${package_name})/meshes/${robot_name}/${mesh}" />
         </geometry>
         <material name="white" />

File: urdf/mobile_robot.urdf.xacro (robot description, xacro)
@@ -33,4 +33,38 @@
                       base_props="${base_props}">
   </xacro:wheel>
+  <gazebo>
+    <plugin name="joint_states" filename="libgazebo_ros_joint_state_publisher.so">
+      <ros>
+        <!-- <namespace>/</namespace> -->
+          <argument>--ros-args</argument>
+          <argument>-r </argument>
+          <argument>~/out:=joint_states</argument>
+      </ros>
+      <update_rate>50</update_rate>
+      <joint_name>back_right_wheel_joint</joint_name>
+      <joint_name>back_left_wheel_joint</joint_name>
+    </plugin>
+    <plugin name="hoverboard_diff_drive" filename="libgazebo_ros_diff_drive.so">
+        <ros>
+          <!-- <namespace>/sim</namespace> -->
+          <remapping>cmd_vel:=/cmd_vel</remapping>
+        </ros>
+      <update_rate>50</update_rate>
+      <left_joint>back_left_wheel_joint</left_joint>
+      <right_joint>back_right_wheel_joint</right_joint>
+      <wheel_separation>0.073</wheel_separation>
+      <wheel_diameter>${back_wheel_props['wheel']['radius']}</wheel_diameter>
+      <command_topic>cmd_vel</command_topic>
+      <!-- output -->
+      <publish_odom>true</publish_odom>
+      <publish_odom_tf>true</publish_odom_tf>
+      <publish_wheel_tf>true</publish_wheel_tf>
+      <odometry_topic>odom</odometry_topic>
+      <odometry_frame>odom</odometry_frame>
+      <robot_base_frame>base_link</robot_base_frame>
+      <max_wheel_torque>30</max_wheel_torque>
+      <max_wheel_acceleration>1.0</max_wheel_acceleration>
+    </plugin>
+  </gazebo>
   <!-- <xacro:include filename="$(find mobile_description)/urdf/mobile_robot_gazebo_plugins.xacro"/>  -->
 </robot>

File: urdf/quimera_robot.gazebo.xacro (robot description, xacro)
@@ -2,9 +2,43 @@
 <robot xmlns:xacro="http://ros.org/wiki/xacro">
   <!-- ros_control plugin -->
-  <gazebo>
+  <!-- <gazebo>
     <plugin name="gazebo_ros_control" filename="libgazebo_ros_control.so">
       <robotNamespace>/quimera_robot</robotNamespace>
-      <!--robotParam>/robot_description</robotParam-->
+      <robotParam>/robot_description</robotParam>
       <robotSimType>gazebo_ros_control/DefaultRobotHWSim</robotSimType>
+    </plugin>
+  </gazebo> -->
+  <gazebo>
+    <plugin name="joint_states" filename="libgazebo_ros_joint_state_publisher.so">
+      <ros>
+        <!-- <namespace>/</namespace> -->
+          <argument>--ros-args</argument>
+          <argument>-r </argument>
+          <argument>~/out:=joint_states</argument>
+      </ros>
+      <update_rate>50</update_rate>
+      <joint_name>back_right_wheel_joint</joint_name>
+      <joint_name>back_left_wheel_joint</joint_name>
+    </plugin>
+    <plugin name="hoverboard_diff_drive" filename="libgazebo_ros_diff_drive.so">
+        <ros>
+          <!-- <namespace>/sim</namespace> -->
+          <remapping>cmd_vel:=/cmd_vel</remapping>
+        </ros>
+      <update_rate>50</update_rate>
+      <left_joint>back_left_wheel_joint</left_joint>
+      <right_joint>back_right_wheel_joint</right_joint>
+      <wheel_separation>0.073</wheel_separation>
+      <wheel_diameter>0.053</wheel_diameter>
+      <command_topic>cmd_vel</command_topic>
+      <!-- output -->
+      <publish_odom>true</publish_odom>
+      <publish_odom_tf>true</publish_odom_tf>
+      <publish_wheel_tf>true</publish_wheel_tf>
+      <odometry_topic>odom</odometry_topic>
+      <odometry_frame>odom</odometry_frame>
+      <robot_base_frame>base_link</robot_base_frame>
+      <max_wheel_torque>30</max_wheel_torque>
+      <max_wheel_acceleration>1.0</max_wheel_acceleration>
     </plugin>
   </gazebo>

Commit message: adjust find mesh file and laserscan plugin

File: urdf/include/common_macros.urdf.xacro (robot description, xacro)
@@ -87,5 +87,5 @@
             <origin xyz="0 0 ${-wheel_props['base']['size']['z']/2.0}" rpy="0 0 0" />
             <geometry>
-                <mesh filename="package://${package_name}/meshes/${robot_name}/${wheel_props['base']['mesh']}" />
+                <mesh filename="file://$(find ${package_name})/meshes/${robot_name}/${wheel_props['base']['mesh']}" />
             </geometry>
             <!-- xacro:insert_block name="material_silver" / TODO use this block? -->
@@ -134,5 +134,5 @@
           <origin xyz="0 0 ${-wheel_props['hub']['size']['z']/2.0}" rpy="0 0 0" />
           <geometry>
-            <mesh filename="file://${package_name}/meshes/${robot_name}/${wheel_props['hub']['mesh']}" />
+            <mesh filename="file://$(find ${package_name})/meshes/${robot_name}/${wheel_props['hub']['mesh']}" />
           </geometry>
           <!-- xacro:insert_block name="material_silver" / TODO use this block? -->
@@ -178,5 +178,5 @@
           <origin xyz="0 0 0" rpy="0 0 0" />
           <geometry>
-            <mesh filename="package://${package_name}/meshes/${robot_name}/${wheel_props['wheel']['mesh']}" />
+            <mesh filename="file://$(find ${package_name})/meshes/${robot_name}/${wheel_props['wheel']['mesh']}" />
           </geometry>
           <!-- TODO use this?: xacro:insert_block name="material_dark_grey" /-->

File: urdf/include/common_sensors.xacro (robot description, xacro)
@@ -12,5 +12,5 @@
         <origin xyz="0 0 0" rpy="0 0 0"/>
         <geometry>
-          <mesh filename="package://${package_name}/meshes/sensors/hokuyo.dae" />
+          <mesh filename="file://$(find ${package_name})/meshes/sensors/hokuyo.dae" />
         </geometry>
       </visual>
@@ -57,8 +57,11 @@
         </noise>
       </ray>
-      <plugin name="gazebo_ros_head_hokuyo_controller" filename="libgazebo_ros_gpu_laser.so">
-        <topicName>/${robot_name}/scan</topicName>
-        <frameName>hokuyo_link</frameName>
-      </plugin>
+      <plugin name="laserscan" filename="libgazebo_ros_ray_sensor.so">
+            <ros>
+              <namespace>/</namespace>
+              <remapping>~/out:=laserscan</remapping>
+            </ros>
+            <output_type>sensor_msgs/LaserScan</output_type>
+          </plugin>
     </sensor>
   </gazebo>
