Commit message: add dependency and adjust base_link color

File: urdf/include/common_sensors.xacro (robot description, xacro)
@@ -31,5 +31,5 @@
     <sensor type="gpu_ray" name="head_hokuyo_sensor">
       <pose>0 0 0 0 0 0</pose>
-      <visualize>true</visualize>
+      <visualize>false</visualize>
       <update_rate>40</update_rate>
       <ray>

File: urdf/quimera_robot.gazebo.xacro (robot description, xacro)
@@ -45,4 +45,7 @@
     </plugin>
   </gazebo>
+  <gazebo reference="base_link">
+    <material>Gazebo/White</material>
+  </gazebo>
   <!-- xacro to set the friction for the wheel. This patch was taken from the MIR
   repository.

Commit message: Add visualize parameter

File: urdf/include/common_sensors.xacro (robot description, xacro)
@@ -1,5 +1,5 @@
 <?xml version="1.0"?>
 <robot xmlns:xacro="http://www.ros.org/wiki/xacro">
-<xacro:macro name="hokuyo_sensor" params=" *joint_origin parent_link ">
+<xacro:macro name="hokuyo_sensor" params=" *joint_origin parent_link visualize">
   <link name="hokuyo_link">
       <collision>
@@ -31,5 +31,5 @@
     <sensor type="gpu_ray" name="head_hokuyo_sensor">
       <pose>0 0 0 0 0 0</pose>
-      <visualize>false</visualize>
+      <visualize>${visualize}</visualize>
       <update_rate>40</update_rate>
       <ray>

File: urdf/quimera_robot.urdf.xacro (robot description, xacro)
@@ -40,5 +40,5 @@
   </xacro:wheel>
   <!-- Sensors -->
-  <xacro:hokuyo_sensor parent_link="base_link" >
+  <xacro:hokuyo_sensor parent_link="base_link" visualize="false">
     <origin xyz="-0.02 0 ${base_props['base']['z_size'] + 0.05}" rpy="0 0 0" />
   </xacro:hokuyo_sensor>

Commit message: Add camera_sensor

File: urdf/include/common_sensors.xacro (robot description, xacro)
@@ -67,3 +67,71 @@
   </gazebo>
 </xacro:macro>
+<xacro:macro name="camera_sensor" params=" *joint_origin parent_link visualize">
+  <link name="camera_link">
+      <collision>
+         <origin xyz="0 0 0" rpy="0 0 0"/>
+        <geometry>
+          <cylinder radius="0.03" length="0.03"/>
+        </geometry>
+      </collision>
+      <visual>
+        <origin xyz="0 0 0" rpy="0 1.57 0"/>
+        <geometry>
+          <cylinder radius="0.01" length="0.01"/>
+        </geometry>
+      </visual>
+      <inertial>
+        <mass value="1e-5" />
+        <origin xyz="0 0 0" rpy="0 0 0"/>
+        <inertia ixx="1e-6" ixy="0" ixz="0" iyy="1e-6" iyz="0" izz="1e-6" />
+      </inertial>
+  </link>
+  <gazebo reference="camera_link">
+    <material>Gazebo/Red</material>
+  </gazebo>
+  <joint name="camera_joint" type="fixed">
+    <axis xyz="0 1 0" />
+    <xacro:insert_block name="joint_origin" />
+    <parent link="${parent_link}"/>
+    <child link="camera_link"/>
+  </joint>
+  <gazebo reference="camera_link">
+    <sensor type="camera" name="camera1">
+      <update_rate>60</update_rate>
+      <visualize>${visualize}</visualize>
+      <camera>
+        <horizontal_fov>1.92</horizontal_fov>
+        <image>
+          <width>640</width>
+          <height>480</height>
+          <format>B8G8R8</format>
+        </image>
+        <depth_camera>
+        </depth_camera>
+        <clip>
+          <near>0.02</near>
+          <far>300</far>
+        </clip>
+        <noise>
+          <type>gaussian</type>
+          <!-- Noise is sampled independently per pixel on each frame.
+                That pixel's noise value is added to each of its color
+                channels, which at that point lie in the range [0,1]. -->
+          <mean>0.0</mean>
+          <stddev>0.007</stddev>
+        </noise>
+      </camera>
+      <plugin name="camera_controller" filename="libgazebo_ros_camera.so">
+        <ros>
+          <!-- <namespace>/</namespace> -->
+          <!-- topics need to be prefixed with camera_name for remapping -->
+          <!-- <remapping>image_raw:=image_demo</remapping> -->
+        </ros>
+        <!-- omit camera_name to default to sensor name -->
+        <!-- <camera_name>mycamera</camera_name> -->
+        <!-- frame_name>omit so it defaults to link name</frame_name-->
+      </plugin>
+    </sensor>
+  </gazebo>
+</xacro:macro>
 </robot>

File: urdf/quimera_robot.urdf.xacro (robot description, xacro)
@@ -40,11 +40,9 @@
   </xacro:wheel>
   <!-- Sensors -->
-  <xacro:hokuyo_sensor parent_link="base_link" visualize="false">
+  <xacro:hokuyo_sensor parent_link="base_link" visualize="true">
     <origin xyz="-0.02 0 ${base_props['base']['z_size'] + 0.05}" rpy="0 0 0" />
   </xacro:hokuyo_sensor>
-  <!-- <xacro:generic_camera name="camera" parent="base_link" ros_topic="image_raw"
-                        cam_info_topic="camera_info" update_rate="30"
-                        res_x="800" res_y="800" image_format="R8G8B8" h_fov="1.4" >
-        <origin xyz="0 0 0" rpy="0 0 0" />
-  </xacro:generic_camera>                       -->
+  <xacro:camera_sensor parent_link="base_link" visualize="true">
+    <origin xyz="0.02 0 ${base_props['base']['z_size']}" rpy="0 0 0" />
+  </xacro:camera_sensor>
 </robot>

Commit message: Add imu sensor

File: urdf/include/common_sensors.xacro (robot description, xacro)
@@ -135,3 +135,48 @@
   </gazebo>
 </xacro:macro>
+<xacro:macro name="imu_sensor" params=" *joint_origin parent_link">
+  <link name="imu_link">
+      <collision>
+         <origin xyz="0 0 0" rpy="0 0 0"/>
+        <geometry>
+          <box size="0.01 0.01 0.01"/>
+        </geometry>
+      </collision>
+      <visual>
+        <origin xyz="0 0 0" rpy="0 0 0"/>
+        <geometry>
+          <box size="0.01 0.01 0.01"/>
+        </geometry>
+      </visual>
+      <inertial>
+        <mass value="1e-5" />
+        <origin xyz="0 0 0" rpy="0 0 0"/>
+        <inertia ixx="1e-6" ixy="0" ixz="0" iyy="1e-6" iyz="0" izz="1e-6" />
+      </inertial>
+  </link>
+  <gazebo reference="imu_link">
+    <material>Gazebo/Yellow</material>
+  </gazebo>
+  <joint name="imu_joint" type="fixed">
+    <axis xyz="0 1 0" />
+    <xacro:insert_block name="joint_origin" />
+    <parent link="${parent_link}"/>
+    <child link="imu_link"/>
+  </joint>
+  <gazebo reference="imu_link">
+    <sensor type="imu" name="my_imu">
+    <always_on>true</always_on>
+    <!-- Publish at 30 hz -->
+    <update_rate>30</update_rate>
+    <plugin name="my_imu_plugin" filename="libgazebo_ros_imu_sensor.so">
+      <ros>
+        <!-- Will publish to /imu/data -->
+        <namespace>/imu</namespace>
+        <argument>~/out:=data</argument>
+      </ros>
+      <!-- frame_name ommited, will be "my_link" -->
+    </plugin>
+    </sensor>
+  </gazebo>
+</xacro:macro>
 </robot>

File: urdf/quimera_robot.urdf.xacro (robot description, xacro)
@@ -40,9 +40,12 @@
   </xacro:wheel>
   <!-- Sensors -->
-  <xacro:hokuyo_sensor parent_link="base_link" visualize="true">
+  <xacro:hokuyo_sensor parent_link="base_link" visualize="false">
     <origin xyz="-0.02 0 ${base_props['base']['z_size'] + 0.05}" rpy="0 0 0" />
   </xacro:hokuyo_sensor>
-  <xacro:camera_sensor parent_link="base_link" visualize="true">
+  <xacro:camera_sensor parent_link="base_link" visualize="false">
     <origin xyz="0.02 0 ${base_props['base']['z_size']}" rpy="0 0 0" />
   </xacro:camera_sensor>
+  <xacro:imu_sensor parent_link="base_link">
+    <origin xyz="0.0 0.05 ${base_props['base']['z_size'] + 0.01}" rpy="0 0 0" />
+  </xacro:imu_sensor>
 </robot>

Commit message: remove models from package.

File: urdf/include/common_sensors.xacro (robot description, xacro)
@@ -12,5 +12,5 @@
         <origin xyz="0 0 0" rpy="0 0 0"/>
         <geometry>
-          <mesh filename="package://${package_name}/meshes/sensors/hokuyo.dae" />
+          <mesh filename="package://mobile_robot_description/meshes/sensors/hokuyo.dae" />
         </geometry>
       </visual>

File: urdf/mobile_robot.urdf.xacro (robot description, xacro)
@@ -4,4 +4,5 @@
   <xacro:property name="robot_name" value="mobile_robot"/>
   <xacro:include filename="$(find ${package_name})/urdf/include/common_macros.urdf.xacro" />
+  <xacro:include filename="$(find ${package_name})/urdf/quimera_robot.gazebo.xacro" />
   <!-- <xacro:set_package_name /> -->
   <xacro:property name="back_wheel_yaml" value="$(find ${package_name})/config/${robot_name}/back_wheel.yaml" />

File: urdf/quimera_robot.gazebo.xacro (robot description, xacro)
@@ -4,7 +4,8 @@
   <gazebo>
     <plugin name="gazebo_ros_control" filename="libgazebo_ros_control.so">
-      <robotNamespace>/quimera_robot</robotNamespace>
+      <robotNamespace>/mobile_robot</robotNamespace>
       <!--robotParam>/robot_description</robotParam-->
       <robotSimType>gazebo_ros_control/DefaultRobotHWSim</robotSimType>
+      <legacyModeNS>True</legacyModeNS>
     </plugin>
   </gazebo>

Commit message: package sanitization

File: urdf/include/common_sensors.xacro (robot description, xacro)
@@ -12,5 +12,5 @@
         <origin xyz="0 0 0" rpy="0 0 0"/>
         <geometry>
-          <mesh filename="file://$(find ${package_name})/meshes/sensors/hokuyo.dae" />
+          <mesh filename="file://$(find mobile_robot_description)/meshes/sensors/hokuyo.dae" />
         </geometry>
       </visual>
